File: HW/USBC/UGC_USBC.kicad_sch (KiCad schematic)
At the start: 3 parts, among them J1 UJ31-CH-G1-SMT-TR

Commit message: Production files
Parts:
- J1: MP UJ31-CH-G1-SMT-TR -> (none); MPN (none) -> UJ31-CH-G1-SMT-TR
Changed lines of the file:
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@@
       (effects (font (size 1.27 1.27)) (justify bottom) hide)
     )
-    (property "MP" "UJ31-CH-G1-SMT-TR" (at 144.78 119.38 0)
+    (property "MPN" "UJ31-CH-G1-SMT-TR" (at 144.78 119.38 0)
       (effects (font (size 1.27 1.27)) (justify bottom) hide)
     )
