File: HW/Main/UGC_Main.kicad_pcb (KiCad board)
At the start: 2 copper layers, 125.7 x 76.4 mm, 136 parts, among them J1 Rumble, J10 Conn_01x01_Pin, J11 Conn_01x01_Pin, J12 Conn_01x01_Pin, J14 USB4105-GF-A-060, J15 Conn_01x05_Pin, J16 Conn_01x05_Pin, J2 LT, J3 RT, J5 Conn_01x01_Pin, J6 Conn_01x01_Pin, J7 Conn_01x01_Pin, J8 Conn_01x01_Pin, J9 Conn_01x01_Pin, Q1 MMBT3904, Q2 MMBT3904, Q3 BSS138DW, Q4 BSS138DW, Q5 Q_NMOS_GSD, Q6 Q_PMOS_GDS, Q7 Q_NMOS_GSD, SW1 SW_Push, SW10 SW_Push, SW11 SW_Push, SW12 SW_Push, SW13 SW_Push, SW14 TS09-63-25-R-260-SMT, SW2 SW_Push, SW3 SW_Push, SW4 SW_Push, SW5 SW_Push, SW6 GL18_SW, SW7 SW_Push, SW8 SW_Push, SW9 TS09-63-25-R-260-SMT, T1 36-8730, U1 ESP32-PICO-MINI-02, U10 ST_LSM6, U11 BQ25180, U12 CH340K, U13 PI3USB4000A, U6 MCP3002, U7 MCP3002, U8 RP2040, U9 GD25Q80EEIGR, Y1 Crystal_GND3

Commit message: Checkpoint 2
Parts:
- removed C24, C25, C26: .047u, Capacitor_SMD:C_0603_1608Metric_Pad1.08x0.95mm_HandSolder
- removed J15: Conn_01x05_Pin, hhl:molex_5034800540
- removed J16: Conn_01x05_Pin, Connector_PinHeader_2.00mm:PinHeader_1x05_P2.00mm_Vertical
- removed L5, L6, L7, L8: SK6805-EC-15, hhl:SK6805-EC-15
- removed R39: 1k, Resistor_SMD:R_0201_0603Metric
- removed T1: 36-8730, hhl:KS_8730
- removed TP1, TP2, TP3: TestPoint, TestPoint:TestPoint_Pad_D1.5mm
- added D10: CUS08F30, Diode_SMD:D_SOD-323_HandSoldering, F.Cu at (226.2, 98.1)
- added D9: CUS08F30, Diode_SMD:D_SOD-323_HandSoldering, F.Cu at (230.6, 97.6)
- added F2: Fuse, Fuse:Fuse_1206_3216Metric_Pad1.42x1.75mm_HandSolder, F.Cu at (228.4, 98.0)
- added J13: 503480-0640, hhl:5034800640, B.Cu at (271.5, 141.2)
- added J4: Conn_01x06_Pin, Connector_PinHeader_2.00mm:PinHeader_1x06_P2.00mm_Vertical, F.Cu at (278.4, 144.2)
- added TP5: TestPoint, TestPoint:TestPoint_Pad_D1.5mm, F.Cu at (184.7, 97.9)
- added U2, U3: GH39F (Hall SOT23), hhl:GH39F, F.Cu at (177.3, 116.6)
- added U4: XC6222, hhl:SOT-89-5, F.Cu at (229.3, 120.5)
- added U5: ST_LSM6, hhl:LGA14, F.Cu at (206.8, 116.0)
- C23, C4: value .047u -> 2.2uF; footprint Capacitor_SMD:C_0603_1608Metric_Pad1.08x0.95mm_HandSolder -> Capacitor_SMD:C_0603_1608Metric
- C3: value .047u -> 47uF 6.3v; footprint Capacitor_SMD:C_0603_1608Metric_Pad1.08x0.95mm_HandSolder -> Capacitor_Tantalum_SMD:CP_EIA-3216-18_Kemet-A
- J1, J2, J3: moved to F.Cu
- J10, J11, J12, J5, J6, J7, J8, J9, U7: moved to B.Cu
- R3: value 1k -> 10k
- R36, R37, R38, R4: value 1k -> 75k; footprint Resistor_SMD:R_0201_0603Metric -> Resistor_SMD:R_0603_1608Metric
- moved D5 145.1 mm to (244.2, 109.2)
- moved D4 145.1 mm to (244.2, 106.4)
- moved D7 142.2 mm to (240.3, 106.4), turned to 180 degrees
- moved D6 141.5 mm to (240.3, 109.2), turned to 180 degrees
- moved D8 139.8 mm to (243.4, 112.3), turned to -90 degrees
- moved C14 135.5 mm to (233.7, 108.8), turned to -90 degrees
- moved C15 135.3 mm to (233.7, 105.7), turned to 90 degrees
- moved R38 133.0 mm to (240.8, 98.7), turned to 90 degrees
- moved R3 132.1 mm to (230.9, 123.7), turned to 180 degrees
- moved R37 131.3 mm to (239.3, 99.6), turned to -90 degrees
- moved C16 130.9 mm to (229.0, 114.2), turned to 180 degrees
- moved R15 130.0 mm to (232.6, 114.2), turned to 90 degrees
- moved R5 128.7 mm to (229.6, 104.5), turned to 180 degrees
- moved C17 126.7 mm to (230.9, 112.9), turned to -90 degrees
- moved R12 125.5 mm to (228.5, 107.1), turned to -90 degrees
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Connections:
- C16 pad 1: Net-(D2-K) -> +5V
- C23 pad 2: LX -> VBUS_SYS
- C3 pad 1: GND -> +3V3
- C3 pad 2: RX -> GND
- C4 pad 1: GND -> +3V3
- C4 pad 2: RY -> GND
- D2 pad 1: Net-(D2-K) -> +5V
- D2 pad 2: VBUS_PRE -> +5V_PRE
- D4 pad 1: Push_A -> Scan_A
- D4 pad 2: Push_A -> Scan_A
- D4 pad 3: Push_A -> Scan_A
- D4 pad 4: ZL_Pull -> L_Pull
- D4 pad 5: Plus_Pull -> DU_Pull
- D4 pad 6: X_Pull -> A_Pull
- D5 pad 1: Push_A -> Scan_A
- D5 pad 2: Push_B -> Scan_B
- D5 pad 3: Push_B -> Scan_B
- D5 pad 4: SL_Pull -> DL_Pull
- D5 pad 5: Y_Pull -> B_Pull
- D5 pad 6: DU_Pull -> SL_Pull
- D6 pad 1: Push_B -> Scan_B
- D6 pad 2: Push_B -> Scan_B
- D6 pad 3: Push_C -> Scan_C
- D6 pad 4: A_Pull -> X_Pull
- D6 pad 5: DD_Pull -> Plus_Pull
- D6 pad 6: R_Pull -> ZL_Pull
- D7 pad 1: Push_C -> Scan_C
- D7 pad 2: Push_C -> Scan_C
- D7 pad 3: Push_C -> Scan_C
- D7 pad 4: DR_Pull -> RS_B_IN
- D7 pad 5: ZR_Pull -> R_Pull
- D7 pad 6: SR_Pull -> DD_Pull
- D8 pad 1: Push_D -> Scan_D
- D8 pad 2: Push_D -> Scan_D
- D8 pad 3: Push_D -> Scan_D
- D8 pad 4: L_Pull -> ZR_Pull
- D8 pad 5: DL_Pull -> DR_Pull
- D8 pad 6: B_Pull -> Y_Pull
- J1 pad 1: unconnected-(J1-Pin_1-Pad1) -> VBUS_SYS
- J1 pad 2: unconnected-(J1-Pin_2-Pad2) -> RUMBLE-
- J10 pad 1: unconnected-(J10-Pin_1-Pad1) -> N_LATCH
- J11 pad 1: unconnected-(J11-Pin_1-Pad1) -> +5V_PRE
- J12 pad 1: unconnected-(J12-Pin_1-Pad1) -> +3V3_PRE
- J14 pad A4_B9: +5V -> +5V_PRE
- J14 pad B4_A9: +5V -> +5V_PRE
- J2 pad 1: unconnected-(J2-Pin_1-Pad1) -> ZL_Pull
- J2 pad 2: unconnected-(J2-Pin_2-Pad2) -> Pulldown_C
- J3 pad 1: unconnected-(J3-Pin_1-Pad1) -> ZR_Pull
- J3 pad 2: unconnected-(J3-Pin_2-Pad2) -> Pulldown_C
- J5 pad 1: unconnected-(J5-Pin_1-Pad1) -> GND
- J6 pad 1: unconnected-(J6-Pin_1-Pad1) -> N_CLOCK
- J7 pad 1: unconnected-(J7-Pin_1-Pad1) -> D+
- J8 pad 1: unconnected-(J8-Pin_1-Pad1) -> N_DATA
- J9 pad 1: unconnected-(J9-Pin_1-Pad1) -> D-
- JP1 pad 1: BAT_LVL -> +5V
- JP1 pad 2: UART0_TX -> VBUS_SYS
- L2 pad 1: SR_RGB -> Net-(L1-DOUT)
- L3 pad 1: Net-(L1-DOUT) -> Net-(L2-DOUT)
- L4 pad 1: Net-(L2-DOUT) -> Net-(L3-DOUT)
- L4 pad 3: Net-(L4-DOUT) -> SR_RGB
- R3 pad 2: RX -> VBUS_SYS
- R36 pad 1: Net-(U14-VOUT) -> ZL_ANALOG
- R36 pad 2: LX -> +3V3
- R37 pad 1: Net-(U15-VOUT) -> GND
- R37 pad 2: LY -> ZR_ANALOG
- R38 pad 1: Net-(U16-VOUT) -> ZR_ANALOG
- R38 pad 2: RX -> +3V3
- R4 pad 1: Net-(U5-VOUT) -> GND
- R4 pad 2: RY -> ZL_ANALOG
- RV1 pad 1: unconnected-(RV1-V+-Pad1) -> +3V3
- RV1 pad 2: unconnected-(RV1-GND-Pad2) -> ZL_ANALOG
- RV1 pad 3: unconnected-(RV1-Signal-Pad3) -> GND
- RV2 pad 1: unconnected-(RV2-V+-Pad1) -> +3V3
- RV2 pad 2: unconnected-(RV2-GND-Pad2) -> ZR_ANALOG
- RV2 pad 3: unconnected-(RV2-Signal-Pad3) -> GND
- SW1 pad 1: unconnected-(SW1-Pad1) -> Pulldown_A
- SW1 pad 2: unconnected-(SW1-Pad2) -> A_Pull
- SW10 pad 1: unconnected-(SW10-Pad1) -> Pulldown_B
- SW10 pad 2: unconnected-(SW10-Pad2) -> DU_Pull
- SW11 pad 1: unconnected-(SW11-Pad1) -> Pulldown_B
- SW11 pad 2: unconnected-(SW11-Pad2) -> DD_Pull
- SW12 pad 1: unconnected-(SW12-Pad1) -> Pulldown_B
- SW12 pad 2: unconnected-(SW12-Pad2) -> DL_Pull
- SW13 pad 1: unconnected-(SW13-Pad1) -> Pulldown_B
- SW13 pad 2: unconnected-(SW13-Pad2) -> DR_Pull
- SW2 pad 1: unconnected-(SW2-Pad1) -> Pulldown_A
- SW2 pad 2: unconnected-(SW2-Pad2) -> B_Pull
- SW3 pad 1: unconnected-(SW3-Pad1) -> Pulldown_A
- SW3 pad 2: unconnected-(SW3-Pad2) -> X_Pull
- SW4 pad 1: unconnected-(SW4-Pad1) -> Pulldown_A
- SW4 pad 2: unconnected-(SW4-Pad2) -> Y_Pull
- SW5 pad 1: unconnected-(SW5-Pad1) -> Pulldown_D
- SW5 pad 2: unconnected-(SW5-Pad2) -> Plus_Pull
- SW6 pad S1: LS_BUTTON -> Pulldown_D
- SW6 pad S2: LS_BUTTON -> Pulldown_D
- SW6 pad S3: unconnected-(SW6-3-PadS3) -> SL_Pull
- SW6 pad S4: unconnected-(SW6-4-PadS4) -> SL_Pull
- SW7 pad 1: unconnected-(SW7-Pad1) -> Pulldown_C
- SW7 pad 2: unconnected-(SW7-Pad2) -> L_Pull
- SW8 pad 1: unconnected-(SW8-Pad1) -> Pulldown_C
- SW8 pad 2: unconnected-(SW8-Pad2) -> R_Pull
- SW9 pad 2: unconnected-(SW9-Pad2) -> GND
- U11 pad A2: Net-(D2-K) -> +5V
- U8 pad 11: Scan_D -> SPI_RX
- U8 pad 12: Scan_B -> RADC_CS
- U8 pad 13: Push_C -> Scan_D
- U8 pad 14: Push_D -> Scan_C
- U8 pad 15: Scan_A -> Scan_B
- U8 pad 16: BTN_PWR -> Scan_A
- U8 pad 17: USB_SEL -> Pulldown_A
- U8 pad 18: ESP_EN -> Pulldown_B
- U8 pad 2: I2C_SDA -> IMU0_CS
- U8 pad 27: LADC_CS -> Pulldown_C
- U8 pad 28: IMU0_CS -> Pulldown_D
- U8 pad 29: SPI_CK -> N_LATCH_3.3
- U8 pad 3: I2C_SCL -> LADC_CS
- U8 pad 30: SPI_TX -> N_DATA_3.3
- U8 pad 31: SPI_RX -> N_CLOCK_3.3
- U8 pad 32: IMU1_CS -> RGB_OUT
- U8 pad 34: RADC_CS -> I2C_SDA
- U8 pad 35: RGB_OUT -> I2C_SCL
- U8 pad 36: RUMBLE -> USB_EN
- U8 pad 37: R_BRAKE -> USB_SEL
- U8 pad 38: BAT_LVL -> ESP_EN
- U8 pad 39: ZL_ANALOG -> ZR_ANALOG
- U8 pad 4: N_DATA_3.3 -> IMU1_CS
- U8 pad 40: ZR_ANALOG -> BAT_LVL
- U8 pad 41: USB_EN -> ZL_ANALOG
- U8 pad 5: N_CLOCK_3.3 -> RUMBLE
- U8 pad 6: N_LATCH_3.3 -> R_BRAKE
- U8 pad 7: Push_A -> BTN_PWR
- U8 pad 8: Scan_C -> SPI_CK
- U8 pad 9: Push_B -> SPI_TX
Routing:
- net Pulldown_C: track 0.00 -> 198.4 mm, vias 0 -> 9
- net Pulldown_D: track 0.00 -> 182.3 mm, vias 0 -> 7
- net Pulldown_B: track 0.00 -> 128.5 mm, vias 0 -> 10
- net D+: track 0.00 -> 121.5 mm, vias 0 -> 2
- net +3V3: track 0.00 -> 116.2 mm, vias 0 -> 40
- net D-: track 0.00 -> 113.9 mm, vias 0 -> 1
- net +5V_PRE: track 0.00 -> 110.8 mm, vias 0 -> 1
- net SL_Pull: track 0.00 -> 104.3 mm, vias 0 -> 4
- net SPI_RX: track 0.00 -> 102.7 mm, vias 0 -> 4
- net SPI_TX: track 0.00 -> 100.5 mm, vias 0 -> 6
- net Pulldown_A: track 0.00 -> 100.4 mm, vias 0 -> 6
- net SPI_CK: track 0.00 -> 99.8 mm, vias 0 -> 5
- net ZL_Pull: track 0.00 -> 99.8 mm, vias 0 -> 3
- net DL_Pull: track 0.00 -> 85.1 mm, vias 0 -> 4
- net L_Pull: track 0.00 -> 85.0 mm, vias 0 -> 2
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- added copper zone on In1.Cu, net +3V3
- added copper zone on B.Cu, net GND
- added copper zone on F.Cu, net GND
- added copper zone on In2.Cu, net GND
- removed copper zone on B.Cu, net (none)
- removed copper zone on F.Cu, net (none)
Other:
- outline, holes or cut-outs redrawn
- copper layers 2 -> 4

Commit message: Production files
Parts:
- added REF**: HHL_Logo, hhl:HHL_Logo, F.Cu at (173.3, 135.5)
Routing:
- net GND: track 22.0 -> 23.6 mm, vias 9 -> 12
- net D+: track 121.5 -> 120.5 mm
- net D-: track 113.9 -> 113.1 mm
- net +5V_PRE: track 110.8 -> 110.0 mm
- net ESP_TX0: track 29.9 -> 30.7 mm
Other:
- board text added: "+"
- board text added: "GCU v1 Designed by Mitch"

Commit message: Update
- Add initial firmware
- Fix PCB trace for SPI RX pin
Connections:
- U8 pad 11: SPI_RX -> R_BRAKE
- U8 pad 6: R_BRAKE -> SPI_RX
Routing:
- net BTN_PWR: track 52.5 -> 53.4 mm
- net R_BRAKE: track 19.0 -> 19.8 mm
Other:
- board text added: "GCU v1.1 Designed by Mitch"
- board text removed: "GCU v1 Designed by Mitch"
