File: HW/Main-r3/UGC_Main.kicad_sch (KiCad schematic)
At the start: 137 parts, among them J1 SM02B-SURS-TF_LF__SN_, J13 503480-0640, J2 LT, J3 RT, J4 Conn_01x06_Pin, J5 UJ31-CH-G1-SMT-TR, J8 Conn_01x02, J9 Conn_01x02, Q1 MMBT3904, Q2 MMBT3904, Q3 BSS138DW, Q4 BSS138DW, Q5 Q_NMOS_GSD, SW1 1TS026A-1000-0550, SW1 SW_Push, SW10 SW_Push, SW11 SW_Push, SW12 SW_Push, SW13 SW_Push, SW14 TS09-63-25-R-260-SMT, SW17 TS09-63-25-R-260-SMT, SW18 TS09-63-25-R-260-SMT, SW19 TS09-63-25-R-260-SMT, SW2 SW_Push, SW20 TS09-63-25-R-260-SMT, SW3 SW_Push, SW4 SW_Push, SW6 GL18_SW, SW7 SW_Push, SW8 SW_Push, SW9 TS09-63-25-R-260-SMT, U1 ESP32-PICO-MINI-02, U10 ST_LSM6, U11 BQ25180, U12 CH340K, U13 PI3USB4000A, U2 GD25Q80EEIGR, U2 GH39F (Hall SOT23), U3 GH39F (Hall SOT23), U4 TPS630001RCR, U5 ST_LSM6, U6 MCP3002, U7 MCP3002, U8 RP2040, Y1 Crystal_GND3

Commit message: Update revision
Connections:
- net RUMBLE is gone; now on net LRA_HI: U8.5 (GPIO3)
- net R_BRAKE is gone; now on net LRA_HI: U8.11 (GPIO8)
Changed lines of the file:
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@@
 		)
 	)
-	(global_label "RUMBLE"
+	(global_label "LRA_HI"
 		(shape input)
 		(at 388.62 166.37 0)
@@
 		)
 		(property "Intersheetrefs" "${INTERSHEET_REFS}"
-			(at 398.4432 166.4494 0)
+			(at 397.8948 166.37 0)
 			(effects
 				(font
@@
 		)
 	)
-	(global_label "R_BRAKE"
+	(global_label "LRA_LO"
 		(shape input)
 		(at 388.62 179.07 0)
@@
 		)
 		(property "Intersheetrefs" "${INTERSHEET_REFS}"
-			(at 399.2294 179.1494 0)
-			(effects
-				(font
+			(at 398.3181 179.07 0)
+			(effects
+				(font

Commit message: Add cad files
Parts:
- removed SW14, SW17, SW18, SW19, SW20, SW9: TS09-63-25-R-260-SMT, hhl:TS09, symbol hhl:TS09-63-25-R-260-SMT
- added D11, D12, D13, D8: BAS16VY,115, Package_TO_SOT_SMD:SOT-363_SC-70-6, symbol progcc_v3:BAS16VY,115
- added SW14, SW17, SW18, SW19, SW5, SW9: SW_TS-1187A, hhl:TS-1187A-C-E-B, symbol hhl:SW_TS-1187A
Connections:
- net A: now also D1.6 (K), U8.29 (GPIO18), D12.6 (K), D8.6 (K); no longer SW1.1, SW10.1, SW7.1, U8.14 (GPIO11)
- net B: now also D1.5 (K), U8.28 (GPIO17), D12.5 (K), D8.5 (K); no longer SW11.1, SW2.1, SW8.1, U8.13 (GPIO10)
- net BAT_LVL: now also U1.4 (I36); no longer U8.40 (GPIO28_ADC2)
- net BTN_PWR: now also SW5.A, SW5.B
- net C: now also D1.4 (K), U8.27 (GPIO16), D12.4 (K), D8.4 (K); no longer D2.6 (K), SW12.1, SW3.1, U8.18 (GPIO15)
- net D: now also D2.6 (K), U8.18 (GPIO15), D11.6 (K), D13.6 (K); no longer D1.4 (K), J2.2 (Pin_2), SW13.1, SW4.1, U8.17 (GPIO14)
- net E: now also D2.5 (K), U8.17 (GPIO14), D11.5 (K), D13.5 (K); no longer D1.5 (K), J3.2 (Pin_2), R35.2, U8.16 (GPIO13)
- net F: now also D2.4 (K), U8.16 (GPIO13), D11.4 (K), D13.4 (K); no longer D1.6 (K), J8.1 (Pin_1), J9.1 (Pin_1), SW6.S1 (1), SW6.S2 (2), U8.15 (GPIO12)
- net GND: now also SW14.A, SW14.B, SW5.C, SW5.D
- net N_CLOCK_3.3: now also U8.32 (GPIO21); no longer U8.31 (GPIO20)
- net N_DATA_3.3: now also U8.31 (GPIO20); no longer U8.30 (GPIO19)
- net N_LATCH_3.3: now also U8.30 (GPIO19); no longer U8.29 (GPIO18)
- net RGB_OUT: now also U8.39 (GPIO27_ADC1); no longer U8.32 (GPIO21)
- net RP_RUN: now also SW14.C, SW14.D
- net ZR_ANALOG: now also U8.40 (GPIO28_ADC2); no longer U8.39 (GPIO27_ADC1)
- net at D2.2 (A): now also SW8.2
- net at D2.3 (A): now also J3.1 (Pin_1)
- removed net W: D2.1 (A), J2.1 (Pin_1), J3.1 (Pin_1), J9.2 (Pin_2), SW7.2, SW8.2
- removed net X: D1.2 (A), SW10.2, SW11.2, SW12.2, SW13.2, SW6.S3 (3), SW6.S4 (4)
- net Y: no longer names the net of D1.3 (A)
- net Y: now also SW3.2; no longer J8.2 (Pin_2)
- removed net Z: D1.1 (A), R34.1, SW1.2, SW2.2, SW3.2, SW4.2
- new net: D8.3 (A), SW12.2
- new net: D13.3 (A), SW2.2
- new net: D12.2 (A), SW17.C, SW17.D
- new net: D1.2 (A), SW1.2
- new net: D13.1 (A), SW19.C, SW19.D
- new net: D11.1 (A), SW7.2
- new net: D12.3 (A), SW18.C, SW18.D
- new net: D11.3 (A), J2.1 (Pin_1)
- new net: D1.1 (A), J8.1 (Pin_1), R34.1
- new net: D8.1 (A), SW10.2
- new net: D11.2 (A), J9.1 (Pin_1), SW6.S3 (3), SW6.S4 (4)
- new net: D8.2 (A), SW11.2
- new net: D12.1 (A), SW9.C, SW9.D
- new net: D2.1 (A), SW4.2
- new net: D13.2 (A), SW13.2
- new net G: J3.2 (Pin_2), J8.2 (Pin_2), R35.2, SW1.1, SW3.1, SW4.1, SW8.1, U8.15 (GPIO12)
- new net H: J2.2 (Pin_2), J9.2 (Pin_2), SW10.1, SW11.1, SW12.1, SW6.S1 (1), SW6.S2 (2), SW7.1, U8.14 (GPIO11)
- new net I: SW13.1, SW17.A, SW17.B, SW18.A, SW18.B, SW19.A, SW19.B, SW2.1, SW9.A, SW9.B, U8.13 (GPIO10)
Other:
- note removed: "C"
- note removed: "C NET"
- note removed: "D"
- note removed: "D NET"
- note removed: "E"
- note removed: "E NET"
- note removed: "F"
- note removed: "F NET"
- moved on the sheet: D1A, D1B, D1C, D2A, D2B, D2C, J2, J3, J8, J9, R34, R35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

Commit message: Main board update
Use new TMR stick on main board
Parts:
- removed SW6: GL18_SW, hhl:GL18, symbol hhl:GL18_SW
- removed U2, U3: GH39F (Hall SOT23), hhl:GH39F, symbol progcc_v3:GH39F (Hall SOT23)
- added SW6: GL18_SW, hhl:GL1807SYAE, symbol hhl:GL1807SYAE-002
Connections:
- net +3V3: now also SW6.X3 (VCC), SW6.Y3 (VCC)
- net GND: now also SW6.X1 (GND), SW6.Y1 (GND)
- net H: now also SW6.S1 (1), SW6.S2 (2)
- net at R1.1: now also SW6.X2 (X_OUT)
- net LS_BTN_IN: now reaches D11.2 (A), J9.1 (Pin_1)
- net LS_BTN_IN: now also SW6.S3 (3), SW6.S4 (4)
- net at R2.1: now also SW6.Y2 (Y_OUT)
Other:
- note added: "Left Stick Btn"
- note removed: "LS"
- moved on the sheet: C1, C2, D11C, D12A, D12B, D12C, D13A, D13B, D13C, D1A, D1B, D1C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
