File: HW/SubStick/UGC_SubStick.kicad_pcb (KiCad board)
At the start: 2 copper layers, 50.1 x 31 mm, 1 part, among them SW1 GL18_SW

Commit message: Updates
- Stick PCB
- USB C pcb
- trigger PCB
Parts:
- added C1: .047u, Capacitor_SMD:C_0603_1608Metric_Pad1.08x0.95mm_HandSolder, F.Cu at (248.3, 161.1)
- added C2: .047u, Capacitor_SMD:C_0603_1608Metric_Pad1.08x0.95mm_HandSolder, F.Cu at (258.1, 145.9)
- added J1: Conn_01x06_Pin, Connector_PinHeader_2.00mm:PinHeader_1x06_P2.00mm_Vertical, F.Cu at (280.8, 140.9)
- added J2: 503480-0640, hhl:5034800640, B.Cu at (278.0, 137.4)
- added R1: 1k, Resistor_SMD:R_0201_0603Metric, F.Cu at (248.9, 160.0)
- added R2: 1k, Resistor_SMD:R_0201_0603Metric, F.Cu at (257.6, 148.4)
- added U1, U2: GH39F (Hall SOT23), hhl:GH39F, F.Cu at (247.2, 149.7)
Connections:
- SW1 pad S1: unconnected-(SW1-1-PadS1) -> RS_B_OUT
- SW1 pad S2: unconnected-(SW1-2-PadS2) -> RS_B_OUT
- SW1 pad S3: unconnected-(SW1-3-PadS3) -> RS_B_IN
- SW1 pad S4: unconnected-(SW1-4-PadS4) -> RS_B_IN
Routing:
- net +3V3: track 0.00 -> 64.0 mm, vias 0 -> 3
- net RS_B_OUT: track 0.00 -> 62.8 mm, vias 0 -> 1
- net RS_B_IN: track 0.00 -> 62.7 mm, vias 0 -> 3
- net RX: track 0.00 -> 57.5 mm, vias 0 -> 1
- net RY: track 0.00 -> 42.5 mm, vias 0 -> 1
- net Net-(U1-VOUT): track 0.00 -> 1.39 mm
- net Net-(U2-VOUT): track 0.00 -> 1.35 mm
- net GND: track 0.00 -> 0.72 mm, vias 0 -> 2
- added copper zone on B.Cu, net GND
- added copper zone on F.Cu, net GND
- removed copper zone on B.Cu, net (none)
- removed copper zone on F.Cu, net (none)
Other:
- outline, holes or cut-outs redrawn

Commit message: R4 updates to hardware
Parts:
- removed U1, U2: GH39F (Hall SOT23), hhl:GH39F
- SW1: footprint hhl:GL18 -> hhl:GL1807SYAE
- moved C1 0.41 mm to (248.2, 161.5)
- moved R1 0.39 mm to (248.7, 160.3)
- moved R2 0.27 mm to (257.8, 148.6)
Connections:
- R1 pad 1: Net-(U1-VOUT) -> Net-(SW1-X_OUT)
- R2 pad 1: Net-(U2-VOUT) -> Net-(SW1-Y_OUT)
Routing:
- net +3V3: track 64.0 -> 56.6 mm, vias 3 -> 0
- net Net-(SW1-X_OUT): track 0.00 -> 2.42 mm
- net Net-(SW1-Y_OUT): track 0.00 -> 2.25 mm
- net Net-(U1-VOUT): track 1.39 -> 0.00 mm
- net Net-(U2-VOUT): track 1.35 -> 0.00 mm
- net RX: track 57.5 -> 58.3 mm
- net RY: track 42.5 -> 41.8 mm
- net GND: track 0.72 -> 1.29 mm, vias 2 -> 5
