File: HW/Main_R4/UGC_Main.kicad_pcb (KiCad board)
At the start: 4 copper layers, 125.7 x 76.4 mm, 142 parts, among them J1 SM02B-SURS-TF_LF__SN_, J13 503480-0640, J2 LT, J3 RT, J4 Conn_01x06_Pin, J5 UJ31-CH-G1-SMT-TR, J6 Trigger, J7 Trigger, J8 Conn_01x02, J9 Conn_01x02, Q1 MMBT3904, Q2 MMBT3904, Q3 BSS138DW, Q4 BSS138DW, Q5 Q_NMOS_GSD, SW1 SW_Push, SW10 SW_Push, SW11 SW_Push, SW12 SW_Push, SW13 SW_Push, SW14 SW_TS-1187A, SW15 1TS026A-1000-0550, SW16 1TS026A-1000-0550, SW17 SW_TS-1187A, SW18 SW_TS-1187A, SW19 SW_TS-1187A, SW2 SW_Push, SW3 SW_Push, SW4 SW_Push, SW5 SW_TS-1187A, SW6 GL18_SW, SW7 SW_Push, SW8 SW_Push, SW9 SW_TS-1187A, U1 ESP32-PICO-MINI-02, U10 ST_LSM6, U11 BQ25180, U12 CH340K, U13 PI3USB4000A, U4 TPS630001RCR, U5 ST_LSM6, U6 MCP3002, U7 MCP3002, U8 RP2040, U9 GD25Q80EEIGR, Y1 Crystal_GND3

Commit message: Update PCB r4
Parts:
- removed D3, D6, D7: M7C, Diode_SMD:D_SOD-523
- removed Q5: Q_NMOS_GSD, Package_TO_SOT_SMD:SOT-23
- removed R31: 10k, Resistor_SMD:R_0201_0603Metric
- removed R32: 100R, Resistor_SMD:R_0201_0603Metric
- removed R33: 0R, Resistor_SMD:R_0201_0603Metric
- added C28: 100n, Capacitor_SMD:C_0201_0603Metric, F.Cu at (227.7, 127.7)
- added C29: 1uF, Capacitor_SMD:C_0201_0603Metric, F.Cu at (230.8, 125.6)
- added C30: 1uF, Capacitor_SMD:C_0201_0603Metric, F.Cu at (229.5, 129.9)
- added C31: 1u, Capacitor_SMD:C_0201_0603Metric, F.Cu at (166.9, 137.1)
- added J10: SM02B-SURS-TF_LF__SN_, hhl:JST_SM02B-SURS-TF_LF__SN_, B.Cu at (166.0, 139.6)
- added R39: 1k, Resistor_SMD:R_0201_0603Metric, F.Cu at (226.5, 127.4)
- added R40: 1.2k, Resistor_SMD:R_0201_0603Metric, F.Cu at (226.9, 128.5)
- added R41: 10k, Resistor_SMD:R_0201_0603Metric, F.Cu at (229.4, 125.6)
- added TP3: TestPoint, TestPoint:TestPoint_Pad_2.0x2.0mm, B.Cu at (163.9, 139.1)
- added TP4: TestPoint, TestPoint:TestPoint_Pad_2.0x2.0mm, B.Cu at (168.0, 139.1)
- added U2: DRV2605LYZFR, Package_BGA:Texas_DSBGA-9_1.4715x1.4715mm_Layout3x3_P0.5mm, F.Cu at (230.5, 127.7)
- C25, C26: moved to F.Cu
- C27: value 100nF -> 1u; moved to F.Cu
- moved TP2 67.6 mm to (280.2, 139.1)
- moved C26 62.8 mm to (279.7, 138.3)
- moved J1 61.1 mm to (278.4, 139.6), turned to 180 degrees
- moved C25 57.0 mm to (277.0, 138.3), turned to 0 degrees
- moved TP1 56.1 mm to (276.6, 139.1)
- moved C27 51.0 mm to (165.2, 137.1)
- moved J3 0.15 mm to (279.7, 133.2)
Connections:
- C27 pad 1: LRA_HI -> GND
- C27 pad 2: GND -> LRA+
Routing:
- net LRA+: track 14.1 -> 139.1 mm, vias 0 -> 3
- net LRA-: track 16.1 -> 139.8 mm, vias 0 -> 3
- net I2C_SCL: track 38.7 -> 60.6 mm, vias 3 -> 5
- net I2C_SDA: track 34.6 -> 56.2 mm, vias 3 -> 5
- net +3V3: track 124.9 -> 134.5 mm, vias 44 -> 51
- net LRA_HI: track 33.7 -> 26.9 mm, vias 2 -> 3
- net GND: track 46.7 -> 51.0 mm, vias 28 -> 56
- net LRA_FILTERED: track 0.00 -> 4.15 mm
- net Net-(U2-EN): track 0.00 -> 1.82 mm
- net Net-(U2-REG): track 0.00 -> 1.68 mm
- net Net-(Q5-G): track 1.57 -> 0.00 mm
- net ABXY_RGB: track 34.2 -> 33.0 mm
- net Net-(D13C-A): track 49.1 -> 48.2 mm
Other:
- outline, holes or cut-outs redrawn
