File: HW/Main_R4/UGC_Main.kicad_sch (KiCad schematic)
At the start: 141 parts, among them J1 SM02B-SURS-TF_LF__SN_, J13 503480-0640, J2 LT, J3 RT, J4 Conn_01x06_Pin, J5 UJ31-CH-G1-SMT-TR, J6 Trigger, J7 Trigger, J8 Conn_01x02, J9 Conn_01x02, Q1 MMBT3904, Q2 MMBT3904, Q3 BSS138DW, Q4 BSS138DW, Q5 Q_NMOS_GSD, SW1 1TS026A-1000-0550, SW1 SW_Push, SW10 SW_Push, SW11 SW_Push, SW12 SW_Push, SW13 SW_Push, SW14 SW_TS-1187A, SW17 SW_TS-1187A, SW18 SW_TS-1187A, SW19 SW_TS-1187A, SW2 SW_Push, SW3 SW_Push, SW4 SW_Push, SW5 SW_TS-1187A, SW6 GL18_SW, SW7 SW_Push, SW8 SW_Push, SW9 SW_TS-1187A, U1 ESP32-PICO-MINI-02, U10 ST_LSM6, U11 BQ25180, U12 CH340K, U13 PI3USB4000A, U2 GD25Q80EEIGR, U4 TPS630001RCR, U5 ST_LSM6, U6 MCP3002, U7 MCP3002, U8 RP2040, Y1 Crystal_GND3

Commit message: Update PCB r4
Parts:
- removed D3, D6, D7: M7C, Diode_SMD:D_SOD-523, symbol Device:D_Schottky
- removed Q5: Q_NMOS_GSD, Package_TO_SOT_SMD:SOT-23, symbol Device:Q_NMOS_GSD
- removed R31: 10k, Resistor_SMD:R_0201_0603Metric, symbol Device:R
- removed R32: 100R, Resistor_SMD:R_0201_0603Metric, symbol Device:R
- removed R33: 0R, Resistor_SMD:R_0201_0603Metric, symbol Device:R
- added C28: 100n, Capacitor_SMD:C_0201_0603Metric, symbol Device:C
- added C29, C30: 1uF, Capacitor_SMD:C_0201_0603Metric, symbol Device:C
- added C31: 1u, Capacitor_SMD:C_0201_0603Metric, symbol Device:C
- added J10: SM02B-SURS-TF_LF__SN_, hhl:JST_SM02B-SURS-TF_LF__SN_, symbol hhl:SM02B-SURS-TF_LF__SN_
- added R39: 1k, Resistor_SMD:R_0201_0603Metric, symbol Device:R
- added R40: 1.2k, Resistor_SMD:R_0201_0603Metric, symbol Device:R
- added R41: 10k, Resistor_SMD:R_0201_0603Metric, symbol Device:R
- added TP3, TP4: TestPoint, TestPoint:TestPoint_Pad_2.0x2.0mm, symbol Connector:TestPoint
- added U2: DRV2605LYZFR, Package_BGA:Texas_DSBGA-9_1.4715x1.4715mm_Layout3x3_P0.5mm, symbol hhl:DRV2605LYZFR
- C27: value 100nF -> 1u
- J8, J9: now not fitted; now left out of the parts list
Connections:
- net +3V3: now also C30.1, R41.2, U2.C2 (VDD)
- net GND: now also C27.1, C28.1, C29.1, C30.2, C31.2, J10.S1 (SHIELD), J10.S2 (SHIELD), R40.1, U2.B3 (GND); no longer C27.2
- net I2C_SCL: now also U2.C1 (SCL)
- net I2C_SDA: now also U2.B2 (SDA)
- net LRA+: now also C27.2, J10.2, TP3.1, U2.A3 (OUT+)
- net LRA-: now also C31.1, J10.1, TP4.1, U2.C3 (OUT-)
- net LRA_HI: now also R39.2; no longer C27.1
- new net: R41.1, U2.A1 (EN)
- new net: C29.2, U2.A2 (REG)
- new net LRA_FILTERED: C28.2, R39.1, R40.2, U2.B1 (IN/TRIG)
Other:
- note removed: "Hall Sensors"
- moved on the sheet: C1, C2, C25, C26, J1, J5, L1, L10, L11, L12, L13, L2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
