File: HW/Main_R4/UGC_Main_R4.kicad_pcb (KiCad board)
At the start: 4 copper layers, 125.7 x 76.4 mm, 153 parts, among them J1 SM02B-SURS-TF_LF__SN_, J10 SM02B-SURS-TF_LF__SN_, J13 503480-0640, J4 Conn_01x06_Pin, J5 UJ31-CH-G1-SMT-TR, J6 Trigger, J7 Trigger, J8 Conn_01x02, J9 Conn_01x02, Q1 MMBT3904, Q2 MMBT3904, Q3 BSS138DW, Q4 BSS138DW, Q5 MMBT2222A, Q6 MMBT2222A, SW1 SW_Push, SW10 SW_Push, SW11 SW_Push, SW12 SW_Push, SW13 SW_Push, SW14 SW_TS-1187A, SW15 1TS026A-1000-0550, SW16 1TS026A-1000-0550, SW17 SW_TS-1187A, SW18 SW_TS-1187A, SW19 SW_TS-1187A, SW2 SW_Push, SW3 SW_Push, SW4 SW_Push, SW5 SW_TS-1187A, SW6 GL18_SW, SW7 SW_Push, SW8 SW_Push, SW9 SW_TS-1187A, U1 ESP32-PICO-MINI-02, U10 ST_LSM6, U11 BQ25180, U12 CH340K, U13 PI3USB4000A, U4 TPS630001RCR, U5 ST_LSM6, U6 MCP3002, U7 MCP3002, U8 RP2040, U9 GD25Q80EEIGR, Y1 Crystal_GND3

Commit message: Update HW
Parts:
- RV1, RV2: footprint hhl:GCC_Slider -> hhl:GCC_Slider_MillMax
- moved R37 1.02 mm to (239.3, 98.6)
- moved R38 0.61 mm to (240.8, 98.1)
- moved R36 0.59 mm to (189.2, 98.0)
- moved R4 0.59 mm to (190.8, 98.0)
- moved C19 0.18 mm to (198.0, 101.6)
Routing:
- net ZR_ANALOG: track 29.4 -> 27.8 mm
- net ZL_ANALOG: track 42.8 -> 43.4 mm
