File: HW/Main_R4/UGC_Main_R4.kicad_sch (KiCad schematic)
At the start: 152 parts, among them J1 SM02B-SURS-TF_LF__SN_, J10 SM02B-SURS-TF_LF__SN_, J13 503480-0640, J4 Conn_01x06_Pin, J5 UJ31-CH-G1-SMT-TR, J6 Trigger, J7 Trigger, J8 Conn_01x02, J9 Conn_01x02, Q1 MMBT3904, Q2 MMBT3904, Q3 BSS138DW, Q4 BSS138DW, Q5 MMBT2222A, Q6 MMBT2222A, SW1 1TS026A-1000-0550, SW1 SW_Push, SW10 SW_Push, SW11 SW_Push, SW12 SW_Push, SW13 SW_Push, SW14 SW_TS-1187A, SW17 SW_TS-1187A, SW18 SW_TS-1187A, SW19 SW_TS-1187A, SW2 SW_Push, SW3 SW_Push, SW4 SW_Push, SW5 SW_TS-1187A, SW6 GL18_SW, SW7 SW_Push, SW8 SW_Push, SW9 SW_TS-1187A, U1 ESP32-PICO-MINI-02, U10 ST_LSM6, U11 BQ25180, U12 CH340K, U13 PI3USB4000A, U2 GD25Q80EEIGR, U4 TPS630001RCR, U5 ST_LSM6, U6 MCP3002, U7 MCP3002, U8 RP2040, Y1 Crystal_GND3

Commit message: Update HW
Parts:
- D1, D10, D9: Price (none) -> 0.0449
- D1, D11, D12, D13, D2, D8: Price (none) -> 0.0186
- D14, D15, D16, D3, D6, D7: Price (none) -> 0.0179
- J1, J10: Price None -> 0.1080
- J13: Price (none) -> 0.48
- J5: Price None -> 1.08323
- L1, L10, L11, L12, L13, L2, L3, L4, L6: Price (none) -> 0.0506
- L5: Price (none) -> 0.0208
- Q1, Q2: Price (none) -> 0.0048
- Q3, Q4: Price (none) -> 0.037
- Q5, Q6: Price (none) -> 0.0050
- RV1, RV2: footprint hhl:GCC_Slider -> hhl:GCC_Slider_MillMax; symbol hhl:Slider_GCC-Gamecube_MB -> hhl:Slider_GCC-Gamecube_MillMax_MB; Price (none) -> 0.2624
- SW1: Price (none) -> 0.0458
- SW14, SW17, SW18, SW19, SW5, SW9: Price (none) -> 0.02
- SW6: Price (none) -> 1.90
- SW7, SW8: Price (none) -> 0.082
- U1: Price (none) -> 3.18
- U10, U5: Price (none) -> 0.59
- U11: Price (none) -> 1.23
- U12: Price (none) -> 0.23
- U13: Price (none) -> 0.13
- U2: Price (none) -> 0.22
- U4: Price None -> 0.565
- U6, U7: Price (none) -> 1.11
- U8: Price (none) -> 0.531
- Y1: Price (none) -> 0.2

Commit message: Add press fit insert
Parts:
- added N1, N2, N3, N4, N5, N6: 0630-0-15-15-30-27-10-0, N/A, symbol Connector_Generic:Conn_01x01
