File: HW/MechTrigger_R4/UGC_MechTrigger.kicad_sch (KiCad schematic)
At the start: 3 parts, among them J1 Conn_01x02_Pin, J2 Conn_01x02_Pin, SW1 SW_Push

Commit message: Update HW
Parts:
- SW1: MPN CPG135301D01 -> CPG135301D03; Price (none) -> 0.45
Changed lines of the file:
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@@
 			)
 		)
-		(property "MPN" "CPG135301D01"
+		(property "MPN" "CPG135301D03"
 			(at 240.03 133.35 0)
 			(effects
+				(font
+					(size 1.27 1.27)
+				)
+				(hide yes)
+			)
+		)
+		(property "Price" "0.45"
+			(at 240.03 133.35 0)
+			(effects
