File: HW/Socket_Trigger_Test/socket_test.kicad_pcb (KiCad board)
At the start: 2 copper layers, 29.9 x 26 mm, 3 parts, among them J1 Conn_01x04_Pin

Commit message: Update HW
Other:
- board size 29.9 x 26 mm -> 29.1 x 26 mm
Changed lines of the file:
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@@
 			(at 0 0 180)
 			(size 2.25 3.25)
-			(drill 1.75)
+			(drill 1.651)
 			(layers "*.Cu" "*.Mask")
 			(remove_unused_layers no)
@@
 			(at 2.5 0 180)
 			(size 2.25 3.25)
-			(drill 1.75)
+			(drill 1.651)
 			(layers "*.Cu" "*.Mask")
 			(remove_unused_layers no)
@@
 			(at -2.5 0 180)
 			(size 2.25 3.25)
-			(drill 1.75)
+			(drill 1.651)
 			(layers "*.Cu" "*.Mask")
 			(remove_unused_layers no)
@@
 			(at 0 0 180)
 			(size 2.25 3.25)
-			(drill 1.75)
+			(drill 1.651)
 			(layers "*.Cu" "*.Mask")
 			(remove_unused_layers no)
@@
 			(at 2.5 0 180)
 			(size 2.25 3.25)
-			(drill 1.75)
+			(drill 1.651)
 			(layers "*.Cu" "*.Mask")
 			(remove_unused_layers no)
@@
 			(at -2.5 0 180)
 			(size 2.25 3.25)
-			(drill 1.75)
+			(drill 1.651)
 			(layers "*.Cu" "*.Mask")
 			(remove_unused_layers no)
@@
 	)
 	(gr_rect
-		(start 235.0516 125.0696)
-		(end 264.922 151.0538)
+		(start 235.585 125.0696)
+		(end 264.6934 151.0538)
 		(stroke
 			(width 0.05)
@@
 		(polygon
 			(pts
-				(xy 233.9086 123.9774) (xy 233.7308 151.8412) (xy 268.0462 152.527) (xy 265.8364 123.9266)
-			)
-		)
+				(xy 231.3432 124.4092) (xy 231.1654 152.273) (xy 268.0462 152.527) (xy 265.8364 123.9266)
+			)
+		)
