File: HW/SubStick_R4K/UGC_SubStick_R4K.kicad_sch (KiCad schematic)
At the start: 7 parts, among them J13 503480-0640, J4 Conn_01x06_Pin, SW1 GL18_SW

Commit message: Update PCBs
- Fix BOMs so they reference real part numbers
Parts:
- C1, C2: value .047u -> 47nF; footprint Capacitor_SMD:C_0603_1608Metric_Pad1.08x0.95mm_HandSolder -> Capacitor_SMD:C_0603_1608Metric; LCSC C15849 -> C519554; MPN (none) -> CC0603JRX7R9BB473; Price (none) -> 0.0026
- J13: LCSC (none) -> C3168077
- J4: MPN (none) -> N/A
- R1, R2: LCSC (none) -> C138165; MPN (none) -> RC0201FR-071KL; Price (none) -> 0.0006
Changed lines of the file:
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@@
+			)
+		)
+		(property "LCSC" "C3168077"
+			(at 165.1 111.76 0)
+			(effects
+				(font
+					(size 1.27 1.27)
+				)
+				(hide yes)
 			)
 		)
@@
 			)
 		)
-		(property "Value" ".047u"
+		(property "Value" "47nF"
 			(at 162.179 144.907 0)
 			(effects
@@
 			)
 		)
-		(property "Footprint" "Capacitor_SMD:C_0603_1608Metric_Pad1.08x0.95mm_HandSolder"
+		(property "Footprint" "Capacitor_SMD:C_0603_1608Metric"
 			(at 164.1348 142.24 0)
 			(effects
@@
 			)
 		)
-		(property "LCSC" "C15849"
+		(property "LCSC" "C519554"
 			(at 165.1 146.05 0)
 			(effects
@@
 			)
 		)
-		(property "MPN" ""
+		(property "MPN" "CC0603JRX7R9BB473"
 			(at 165.1 146.05 0)
 			(effects
@@
 		)
 		(property "Manufacturer" ""
+			(at 165.1 146.05 0)
+			(effects
+				(font
+					(size 1.27 1.27)
+				)
+				(hide yes)
+			)
+		)
+		(property "Price" "0.0026"
 			(at 165.1 146.05 0)
 			(effects
@@
 			)
 		)
+		(property "LCSC" "C138165"
+			(at 152.4 139.7 0)
+			(effects
+				(font
+					(size 1.27 1.27)
+				)
+				(hide yes)
+			)
+		)
+		(property "MPN" "RC0201FR-071KL "
+			(at 152.4 139.7 0)
+			(effects
+				(font
+					(size 1.27 1.27)
+				)
+				(hide yes)
+			)
+		)
+		(property "Price" "0.0006"
+			(at 152.4 139.7 0)
+			(effects
+				(font
+					(size 1.27 1.27)
+				)
+				(hide yes)
+			)
+		)
 		(pin "1"
 		)
@@
 			)
 		)
-		(property "Value" ".047u"
+		(property "Value" "47nF"
 			(at 144.399 143.637 0)
 			(effects
@@
 			)
 		)
-		(property "Footprint" "Capacitor_SMD:C_0603_1608Metric_Pad1.08x0.95mm_HandSolder"
+		(property "Footprint" "Capacitor_SMD:C_0603_1608Metric"
 			(at 146.3548 140.97 0)
 			(effects
@@
 			)
 		)
-		(property "LCSC" "C15849"
+		(property "LCSC" "C519554"
 			(at 147.32 144.78 0)
 			(effects
@@
 			)
 		)
-		(property "MPN" ""
+		(property "MPN" "CC0603JRX7R9BB473"
 			(at 147.32 144.78 0)
 			(effects
@@
 		)
 		(property "Manufacturer" ""
+			(at 147.32 144.78 0)
+			(effects
+				(font
+					(size 1.27 1.27)
+				)
+				(hide yes)
+			)
+		)
+		(property "Price" "0.0026"
 			(at 147.32 144.78 0)
 			(effects
@@
 		)
 		(property "Description" "Resistor"
+			(at 170.18 142.24 0)
+			(effects
+				(font
+					(size 1.27 1.27)
+				)
+				(hide yes)
+			)
+		)
+		(property "LCSC" "C138165"
+			(at 170.18 142.24 0)
+			(effects
+				(font
+					(size 1.27 1.27)
+				)
+				(hide yes)
+			)
+		)
+		(property "MPN" "RC0201FR-071KL "
+			(at 170.18 142.24 0)
+			(effects
+				(font
+					(size 1.27 1.27)
+				)
+				(hide yes)
+			)
+		)
+		(property "Price" "0.0006"
 			(at 170.18 142.24 0)
 			(effects
@@
 			(at 115.57 115.57 0)
 			(effects
+				(font
+					(size 1.27 1.27)
+				)
+				(hide yes)
+			)
+		)
+		(property "MPN" "N/A"
+			(at 115.57 115.57 0)
+			(effects
