File: HW/Main_S1/UGC_Main_S1.kicad_sch (KiCad schematic)
At the start: 140 parts, among them J1 SM02B-SURS-TF_LF__SN_, J10 SM02B-SURS-TF_LF__SN_, J13 503480-0640, J2 503480-0640, J4 Conn_01x06_Pin, J5 UJ31-CH-G1-SMT-TR, J6 Trigger, J7 Trigger, J8 Conn_01x02, J9 Conn_01x02, Q3 BSS138DW, Q4 BSS138DW, Q5 MMBT2222A, Q6 MMBT2222A, SW1 1TS026A-1000-0550, SW1 SW_Push, SW10 SW_Push, SW11 SW_Push, SW12 SW_Push, SW13 SW_Push, SW14 SW_TS-1187A, SW17 SW_TS-1187A, SW18 SW_TS-1187A, SW19 SW_TS-1187A, SW2 SW_Push, SW3 SW_Push, SW4 SW_Push, SW5 SW_TS-1187A, SW6 GL18_SW, SW7 SW_Push, SW8 SW_Push, SW9 SW_TS-1187A, U10 ST_LSM6, U2 GD25Q80EEIGR, U4 TPS630001RCR, U6 MCP3002, U7 MCP3002, U8 RP2040, X1 ModConnect, X2 ModConnect, X3 ModConnect, X4 ModConnect, X5 ModConnect, X6 ModConnect, Y1 ABM8-272-T3

Commit message: Update PCBs
- Fix BOMs so they reference real part numbers
Parts:
- removed N1, N2, N3, N4, N5, N6: 0630-0-15-15-30-27-10-0, N/A, symbol Connector_Generic:Conn_01x01
- C1: value 47uF 6.3v -> 47uF; LCSC (none) -> C7190; MPN (none) -> TAJA476K006RNJ; Price (none) -> 0.0544
- C1, C2: value .047u -> 47nF; LCSC C15849 -> C519554; MPN (none) -> CC0603JRX7R9BB473; Price (none) -> 0.0026
- C10, C24, C6: value 100n -> 100nF; footprint Capacitor_SMD:C_0201_0603Metric -> Capacitor_SMD:C_0402_1005Metric; LCSC (none) -> C541406; MPN (none) -> CC0402KRX7R5BB104; Price (none) -> 0.0007
- C10, C5, C7, C9: value 100n -> 100nF; LCSC (none) -> C541406; MPN (none) -> CC0402KRX7R5BB104; Price (none) -> 0.0007
- C12, C13: footprint Capacitor_SMD:C_0603_1608Metric -> Capacitor_SMD:C_0402_1005Metric; LCSC C1525 -> C541406; MPN (none) -> CC0402KRX7R5BB104; Price (none) -> 0.0007
- C14, C15: value 15p -> 15pF; LCSC (none) -> C326803; MPN (none) -> CC0402FRNPO9BN150; Price (none) -> 0.002
- C2, C3: LCSC (none) -> C17024; MPN (none) -> CL21A106KPFNNNE; Price (none) -> 0.0050
- C25, C32: footprint Capacitor_SMD:C_0201_0603Metric -> Capacitor_SMD:C_0402_1005Metric; LCSC (none) -> C541406; MPN (none) -> CC0402KRX7R5BB104; Price (none) -> 0.0007
- C26, C27, C33, C34: value 1u -> 1uF; footprint Capacitor_SMD:C_0201_0603Metric -> Capacitor_SMD:C_0402_1005Metric; LCSC (none) -> C107372; MPN (none) -> CL05A105KQ5NNNC; Price (none) -> 0.0009
- C8: value 1u -> 1uF; LCSC (none) -> C107372; MPN (none) -> CL05A105KQ5NNNC; Price (none) -> 0.0009
- D1, D11, D12, D13, D2, D8: LCSC (none) -> C135826; MPN (none) -> BAS16VY,115
- D10, D9: LCSC (none) -> C27636112; Price 0.0449 -> 0.0092
- J1, J10: LCSC (none) -> C566239
- J13, J2: LCSC (none) -> C3168077; Price 0.48 -> 0.4028
- J4, SW1, SW10, SW11, SW12, SW13, SW2, SW3, SW4, TP1, TP2, TP5, TP6, TP7, X1, X2, X3, X4, X5, X6: MPN (none) -> N/A
- J5: LCSC (none) -> C22359729; Purchase-URL https://www.snapeda.com/api/url_track_click_mouser/?unipart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 -> (none)
- J6, J7, J8, J9: LCSC (none) -> C7499302; MPN (none) -> PH2.0 mm Female; Price (none) -> 0.0098
- L1, L10, L11, L12, L13, L2, L3, L4, L6: LCSC (none) -> C2890035; Price 0.0506 -> 0.0492
- Q5, Q6: LCSC (none) -> C916372; MPN (none) -> MMBT2222A
- R1, R2, R23, R24, R25, R26, R27, R28, R7: footprint Resistor_SMD:R_0201_0603Metric -> Resistor_SMD:R_0402_1005Metric; LCSC (none) -> C106235; MPN (none) -> RC0402FR-071KL; Price (none) -> 0.0004
- R11: value 330 -> 330R; LCSC (none) -> C105875; MPN (none) -> RC0402FR-07330RL; Price (none) -> 0.0005
- R12: LCSC (none) -> C106235; MPN (none) -> RC0402FR-071KL; Price (none) -> 0.0004
- R21, R22: value 5.1kohm -> 5.1k; footprint Resistor_SMD:R_0603_1608Metric -> Resistor_SMD:R_0402_1005Metric; LCSC (none) -> C105872; MPN (none) -> RC0402FR-075K1L; Price (none) -> 0.0004
- R3: value 100 -> 100R; footprint Resistor_SMD:R_0201_0603Metric -> Resistor_SMD:R_0402_1005Metric; LCSC (none) -> C106232; MPN (none) -> RC0402FR-07100RL; Price (none) -> 0.0005
- R31, R39: LCSC C25804 -> C60491; MPN (none) -> RC0402FR-07100KL; Price (none) -> 0.0004
- R32, R40: LCSC C22775 -> C106232; MPN (none) -> RC0402FR-07100RL; Price (none) -> 0.0005
- R33, R41: LCSC C22775 -> C106231; MPN (none) -> RC0402FR-070RL; Price (none) -> 0.0004
- R34, R35: LCSC (none) -> C106231; MPN (none) -> RC0402FR-070RL; Price (none) -> 0.0004
- R36, R37, R38, R4: footprint Resistor_SMD:R_0603_1608Metric -> Resistor_SMD:R_0402_1005Metric; LCSC (none) -> C137935; MPN (none) -> RC0402FR-0775KL; Price (none) -> 0.0004
- R5: footprint Resistor_SMD:R_0201_0603Metric -> Resistor_SMD:R_0402_1005Metric; LCSC (none) -> C60491; MPN (none) -> RC0402FR-07100KL; Price (none) -> 0.0004
- R6, R7: value 27 -> 27R; LCSC (none) -> C490808; MPN (none) -> ERA1AEB103C; Price (none) -> 0.0523
- RV1, RV2: LCSC (none) -> C127475
- S1, S2, S3, S4, S5, S6: LCSC (none) -> C17526581; Price (none) -> 0.754
- SW14, SW17, SW18, SW19, SW5, SW9: LCSC (none) -> C318887; Price 0.02 -> 0.0197
- U4: LCSC (none) -> C28060; Purchase-URL https://www.snapeda.com/api/url_track_click_mouser/?unipart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 -> (none)
- U6, U7: LCSC (none) -> C635958
- U8: LCSC (none) -> C2040
- Y1: LCSC (none) -> C20625731; Price (none) -> 0.2381

Commit message: Fix some wrong MPNs
Parts:
- C14, C15: Price 0.002 -> 0.0022
- R31, R39, R5: LCSC C60491 -> C60490; MPN RC0402FR-07100KL -> RC0402FR-0710KL
- R6, R7: LCSC C490808 -> C273268; MPN ERA1AEB103C -> RC0201FR-0727RL; Price 0.0523 -> 0.0006
Changed lines of the file:
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@@
 			)
 		)
-		(property "LCSC" "C60491"
+		(property "LCSC" "C60490"
 			(at 199.39 359.41 0)
 			(effects
@@
 			)
 		)
-		(property "MPN" "RC0402FR-07100KL "
+		(property "MPN" "RC0402FR-0710KL"
 			(at 199.39 359.41 0)
 			(effects
@@
 			)
 		)
-		(property "Price" "0.002"
+		(property "Price" "0.0022"
 			(at 325.12 212.09 0)
 			(effects
@@
 			)
 		)
-		(property "LCSC" "C490808"
+		(property "LCSC" "C273268"
 			(at 294.64 288.29 0)
 			(effects
@@
 			)
 		)
-		(property "MPN" "ERA1AEB103C"
+		(property "MPN" "RC0201FR-0727RL "
 			(at 294.64 288.29 0)
 			(effects
@@
 			)
 		)
-		(property "Price" "0.0523"
+		(property "Price" "0.0006"
 			(at 294.64 288.29 0)
 			(effects
@@
 			)
 		)
-		(property "LCSC" "C60491"
+		(property "LCSC" "C60490"
 			(at 199.39 304.8 0)
 			(effects
@@
 			)
 		)
-		(property "MPN" "RC0402FR-07100KL "
+		(property "MPN" "RC0402FR-0710KL"
 			(at 199.39 304.8 0)
 			(effects
@@
 			)
 		)
-		(property "LCSC" "C490808"
+		(property "LCSC" "C273268"
 			(at 294.64 285.75 0)
 			(effects
@@
 			)
 		)
-		(property "MPN" "ERA1AEB103C"
+		(property "MPN" "RC0201FR-0727RL "
 			(at 294.64 285.75 0)
 			(effects
@@
 			)
 		)
-		(property "Price" "0.0523"
+		(property "Price" "0.0006"
 			(at 294.64 285.75 0)
 			(effects
@@
 			)
 		)
-		(property "Price" "0.002"
+		(property "Price" "0.0022"
 			(at 325.12 222.25 0)
 			(effects
@@
 			)
 		)
-		(property "LCSC" "C60491"
+		(property "LCSC" "C60490"
 			(at 287.02 278.13 0)
 			(effects
@@
 			)
 		)
-		(property "MPN" "RC0402FR-07100KL "
+		(property "MPN" "RC0402FR-0710KL"
 			(at 287.02 278.13 0)
 			(effects

Commit message: Minor updates to text
Parts:
- added J11: Conn_01x04_Pin, Connector_PinHeader_2.00mm:PinHeader_1x04_P2.00mm_Vertical, symbol Connector:Conn_01x04_Pin
- added J3: Conn_01x06_Pin, Connector_PinHeader_2.00mm:PinHeader_1x06_P2.00mm_Vertical, symbol Connector:Conn_01x06_Pin
Connections:
- net +3V3_PRE: now also J3.1 (Pin_1)
- net D+: now also J11.2 (Pin_2)
- net D-: now also J11.3 (Pin_3)
- net GND: now also J11.4 (Pin_4), J3.4 (Pin_4), J3.5 (Pin_5), J3.6 (Pin_6)
- net N_DATA: now also J3.3 (Pin_3)
- net VBUS_SYS: now also J11.1 (Pin_1), J3.2 (Pin_2)

Commit message: Update PCB directory
Accessory boards have been migrated to Open-GC-Ultimate
Parts:
- removed J11: Conn_01x04_Pin, Connector_PinHeader_2.00mm:PinHeader_1x04_P2.00mm_Vertical, symbol Connector:Conn_01x04_Pin
- removed J3: Conn_01x06_Pin, Connector_PinHeader_2.00mm:PinHeader_1x06_P2.00mm_Vertical, symbol Connector:Conn_01x06_Pin
- removed SW1: 1TS026A-1000-0550, hhl:1TS026A-1000-0550, symbol hhl:1TS026A-1000-0550
- added U1: ST_LSM6, hhl:LGA14, symbol progcc_v3:ST_LSM6
Connections:
- net +3V3: now also U1.5 (VDDIO), U1.8 (VDD)
- net GND: now also U1.2 (SDx), U1.3 (SCx), U1.6 (GNDIO), U1.7 (GND)
- net IMU1_CS: now also U1.12 (CS)
- net RP_RUN: no longer SW14.C, SW14.D
- net SPI_CK: now also U1.13 (SCL)
- net SPI_RX: now also U1.1 (SDO)
- net SPI_TX: now also U1.14 (SDA)
- net USB_BOOT: now also SW14.C, SW14.D
- no-connect marks 4 -> 8
Other:
- note added: "IMU 1"
- moved on the sheet: C10, R7, SW14, U2

Commit message: PCB Production files update
Parts:
- C1, C2: Package (none) -> 0603
- C10, C12, C13, C14, C15, C24, C25, C26, C27, C32, C33, C34, C5, C6, C7, C8, C9, R1, R11, R12, R2, R21, R22, R23, R24, R25, R26, R27, R28, R3, R31, R32, R33, R34, R35, R36, R37, R38, R39, R4, R40, R41, R5, R7: Package (none) -> 0402
- C2, C3: Package (none) -> 0805
- D1, D11, D12, D13, D2, D8: Package (none) -> SOT-363
- D10, D9: Package (none) -> SOD-323
- D14, D15, D16, D3, D6, D7: Package (none) -> SOD-523
- J1, J10: Package None -> SMD,P=0.8mm,Surface Mount，Right Angle
- J13, J2: MPN 503480-0640 -> 5034800640; Package (none) -> SMD,P=0.5mm,Surface Mount，Right Angle
- J5: Package None -> -
- J6, J7: LCSC C7499302 -> C5175230; MPN PH2.0 mm Female -> HDGC2001WV-2P; Package (none) -> Plugin,P=2mm
- J8, J9: LCSC C7499302 -> -; Link (none) -> -; MPN PH2.0 mm Female -> -; Package (none) -> -
- L1, L10, L11, L12, L13, L2, L3, L4, L6: Package (none) -> 0606
- L5: Package (none) -> 1008
- Q3, Q4: Package (none) -> SC-70-6(SOT-363)
- Q5, Q6: Package (none) -> SOT-23
- R6, R7: Package (none) -> 0201
- RV1, RV2: LCSC C127475 -> -; Package (none) -> -; now not fitted
- SW14, SW17, SW18, SW19, SW5, SW9: value SW_TS-1187A -> TS-1187A-C-A-B; Package (none) -> SMD
- U1, U10: Package (none) -> LGA-14(2.5x3)
- U2: Package (none) -> USON-8-EP(2x3)
- U6, U7: Package (none) -> MSOP-8
- U8: Package (none) -> LQFN-56(7x7)
- Y1: Package (none) -> SMD3225-4P

Commit message: Update S1
Parts:
- removed U6, U7: MCP3002, Package_SO:MSOP-8_3x3mm_P0.65mm, symbol Analog_ADC:MCP3002
- added C16: 100nF, Capacitor_SMD:C_0402_1005Metric, symbol Device:C
- added S7: TMUX1204DQAR, hhl:TMUX1204DQAR, symbol hhl:TMUX1204DQAR
- L1, L10, L11, L12, L13, L2, L3, L4, L6: value SK6805-EC-15 -> SK6805-EC-10; footprint hhl:SK6805-EC-15 -> hhl:SK6805-EC-10; symbol progcc_v3:SK6805-EC-15 -> hhl:SK6805-EC-10; MPN SK6805-EC-15 -> SK6805-EC-10
Connections:
- net +3V3: now also C16.1, S7.5 (EN), S7.6 (VDD)
- net GND: now also C16.2, S7.3 (GND)
- net LX: now also S7.2 (S1)
- net LY: now also S7.4 (S3)
- net RX: now also S7.7 (S4)
- net RY: now also S7.9 (S2)
- net ESP_EN renamed ADC_MUX_OUT
- net ADC_MUX_OUT: now also S7.8 (D)
- net I2C_SCL renamed ADC_ADDR_0
- net ADC_ADDR_0: now also S7.1 (A0)
- net I2C_SDA: no longer names the net of U8.34 (GPIO22)
- net LADC_CS: no longer names the net of U8.3 (GPIO1)
- net RADC_CS: no longer names the net of U8.12 (GPIO9)
- net USB_EN renamed ADC_ADDR_1
- net ADC_ADDR_1: now also S7.10 (A1)
- net USB_SEL: no longer names the net of U8.37 (GPIO25)
Other:
- note removed: "ADCs"

Commit message: Update S1 BOM
Parts:
- D10, D9: value CUS08F30 -> CUS08F30,H3F; LCSC C27636112 -> C150183; MPN CUS08F30 -> CUS08F30,H3F
Changed lines of the file:
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@@
 			)
 		)
-		(property "Value" "CUS08F30"
+		(property "Value" "CUS08F30,H3F"
 			(at 273.05 62.23 0)
 			(effects
@@
 			)
 		)
-		(property "MPN" "CUS08F30"
+		(property "MPN" "CUS08F30,H3F"
 			(at 270.51 62.23 0)
 			(effects
@@
 			)
 		)
-		(property "LCSC" "C27636112"
+		(property "LCSC" "C150183"
 			(at 270.51 62.23 0)
 			(effects
@@
 			)
 		)
-		(property "Value" "CUS08F30"
+		(property "Value" "CUS08F30,H3F"
 			(at 318.77 57.15 0)
 			(effects
@@
 			)
 		)
-		(property "MPN" "CUS08F30"
+		(property "MPN" "CUS08F30,H3F"
 			(at 318.77 59.69 0)
 			(effects
@@
 			)
 		)
-		(property "LCSC" "C27636112"
+		(property "LCSC" "C150183"
 			(at 318.77 59.69 0)
 			(effects

Commit message: S1 ESD
Parts:
- added U2, U3, U5: USBLC6-2P6, Package_TO_SOT_SMD:SOT-666, symbol Power_Protection:USBLC6-2P6
Connections:
- net +3V3_PRE: now also U5.5 (VBUS)
- net D+: now also U2.3 (I/O2); no longer R6.1
- net D-: now also U2.1 (I/O1); no longer R7.1
- net GND: now also U2.2 (GND), U3.2 (GND), U5.2 (GND)
- net N_CLOCK: now also U5.3 (I/O2); no longer Q4.6 (D1), R27.2
- net N_DATA: now also U3.6 (I/O1); no longer Q4.4 (S2), R28.2
- net N_LATCH: now also U3.4 (I/O2); no longer Q3.4 (S2), R26.2
- net VBUS_SYS: now also U2.5 (VBUS)
- new net N_CLOCK_SAFE: Q4.6 (D1), R27.2, U5.4 (I/O2)
- new net N_DATA_SAFE: Q4.4 (S2), R28.2, U3.1 (I/O1)
- new net N_LATCH_SAFE: Q3.4 (S2), R26.2, U3.3 (I/O2)
- new net SAFE_D+: R6.1, U2.4 (I/O2)
- new net SAFE_D-: R7.1, U2.6 (I/O1)
Other:
- note added: "ESD"
