File: HW/Main_R5/UGC_Main_R5.kicad_pcb (KiCad board)
At the start: 4 copper layers, 125.7 x 76.4 mm, 168 parts, among them J1 SM02B-SURS-TF_LF__SN_, J10 SM02B-SURS-TF_LF__SN_, J13 503480-0640, J2 503480-0640, J4 Conn_01x06_Pin, J5 UJ31-CH-G1-SMT-TR, J6 Trigger, J7 Trigger, J8 Conn_01x02, J9 Conn_01x02, Q1 MMBT3904, Q2 MMBT3904, Q3 BSS138DW, Q4 BSS138DW, Q5 MMBT2222A, Q6 MMBT2222A, SW1 SW_Push, SW10 SW_Push, SW11 SW_Push, SW12 SW_Push, SW13 SW_Push, SW14 SW_TS-1187A, SW15 1TS026A-1000-0550, SW16 1TS026A-1000-0550, SW17 SW_TS-1187A, SW18 SW_TS-1187A, SW19 SW_TS-1187A, SW2 SW_Push, SW3 SW_Push, SW4 SW_Push, SW5 SW_TS-1187A, SW6 GL18_SW, SW7 SW_Push, SW8 SW_Push, SW9 SW_TS-1187A, U1 ESP32-PICO-MINI-02, U10 ST_LSM6, U11 BQ25180, U12 CH340K, U13 PI3USB4000A, U4 TPS630001RCR, U5 ST_LSM6, U6 MCP3002, U7 MCP3002, U8 RP2040, U9 GD25Q80EEIGR, X1 ModConnect, X2 ModConnect, X3 ModConnect, X4 ModConnect, X5 ModConnect, X6 ModConnect, Y1 ABM8-272-T3

Commit message: R5 Update
Parts:
- removed C19: 10uF, Capacitor_SMD:C_0805_2012Metric
- removed C20, C22: 100nF, Capacitor_SMD:C_0201_0603Metric
- removed C21: 1uF, Capacitor_SMD:C_0201_0603Metric
- removed Q1, Q2: MMBT3904, Package_TO_SOT_SMD:SOT-23
- removed R20, R29, R30: 10k, Resistor_SMD:R_0201_0603Metric
- removed SW16: 1TS026A-1000-0550, hhl:1TS026A-1000-0550
- removed U12: CH340K, hhl:ESSOP-10
- removed U13: PI3USB4000A, Package_DFN_QFN:Texas_UQFN-10_1.5x2mm_P0.5mm
- removed U6, U7: MCP3002, Package_SO:MSOP-8_3x3mm_P0.65mm
- added L14: SK6805-EC-15, hhl:SK6805-EC-15, F.Cu at (199.6, 146.5)
- added L15: SK6805-EC-15, hhl:SK6805-EC-15, F.Cu at (196.2, 143.1)
- added L7: BLM18AG601SN1D, Inductor_SMD:L_0603_1608Metric, F.Cu at (187.3, 69.1)
- added L8: SK6805-EC-15, hhl:SK6805-EC-15, F.Cu at (192.9, 146.5)
- added L9: SK6805-EC-15, hhl:SK6805-EC-15, F.Cu at (196.2, 149.8)
- added P1: RPI-RM2, hhl:RPI_RM2, F.Cu at (205.3, 102.8)
- added S7: TMUX1204DQAR, hhl:TMUX1204DQAR, F.Cu at (187.9, 65.1)
- added U2: USBLC6-2P6, Package_TO_SOT_SMD:SOT-666, F.Cu at (187.3, 57.2)
- added U3: USBLC6-2P6, Package_TO_SOT_SMD:SOT-666, F.Cu at (187.3, 60.6)
- C18: footprint Capacitor_SMD:C_0201_0603Metric -> Capacitor_SMD:C_0402_1005Metric
- D1, D10, D2, D9: value CUS08F30 -> CUS08F30,H3F
- R17: value 10k -> 470R
- R18, R19: value 0R -> 1k
- SW14, SW17, SW18, SW19, SW5, SW9: value SW_TS-1187A -> TS-1187A-C-A-B
- U1: value ESP32-PICO-MINI-02 -> USBLC6-2P6; footprint hhl:MODULE_ESP32-PICO-MINI-02 -> Package_TO_SOT_SMD:SOT-666
- moved R18 51.1 mm to (253.2, 88.1)
- moved R19 47.9 mm to (247.9, 87.0)
- moved R8 38.0 mm to (243.9, 86.9)
- moved U1 28.4 mm to (230.8, 92.2)
- moved C12 3.34 mm to (204.8, 114.1), turned to 180 degrees
- moved R26 1.17 mm to (224.4, 95.3), turned to -90 degrees
- moved D2 0.49 mm to (214.3, 96.5)
Connections:
- L4 pad 3: PLAYER_RGB -> DPAD_RGB
- L6 pad 1: PLAYER_RGB -> Net-(L15-DOUT)
- Q3 pad 4: N_LATCH -> N_LATCH_SAFE
- Q4 pad 4: N_DATA -> N_DATA_SAFE
- Q4 pad 6: N_CLOCK -> N_CLOCK_SAFE
- R16 pad 1: ESP_DTR -> Net-(P1B-IRQ)
- R16 pad 2: Net-(Q1-B) -> WL_D
- R17 pad 1: Net-(Q2-B) -> WL_D
- R17 pad 2: ESP_RTS -> Net-(P1A-DO)
- R18 pad 1: ESP_IO15 -> +3V3
- R18 pad 2: ESP_CTS -> I2C0_SCL
- R19 pad 1: ESP_RTS -> I2C0_SDA
- R19 pad 2: ESP_IO13 -> +3V3
- R26 pad 2: N_LATCH -> N_LATCH_SAFE
- R27 pad 2: N_CLOCK -> N_CLOCK_SAFE
- R28 pad 2: N_DATA -> N_DATA_SAFE
- R6 pad 1: RP_USB+ -> SAFE_D+
- R7 pad 1: RP_USB- -> SAFE_D-
- R8 pad 2: I2C_SCL -> I2C1_SCL
- R9 pad 1: I2C_SDA -> I2C1_SDA
- U1 pad 1: GND -> D-
- U1 pad 3: +3V3 -> D+
- U1 pad 4: BAT_LVL -> SAFE_D+
- U1 pad 5: unconnected-(U1-I37-Pad5) -> VBUS_PRE
- U1 pad 6: unconnected-(U1-I38-Pad6) -> SAFE_D-
- U10 pad 1: SPI_RX -> +3V3
- U10 pad 12: IMU0_CS -> +3V3
- U10 pad 13: SPI_CK -> I2C0_SCL
- U10 pad 14: SPI_TX -> I2C0_SDA
- U5 pad 1: SPI_RX -> GND
- U5 pad 12: IMU1_CS -> +3V3
- U5 pad 13: SPI_CK -> I2C0_SCL
- U5 pad 14: SPI_TX -> I2C0_SDA
- U8 pad 11: LRA_R -> LRA_L
- U8 pad 12: RADC_CS -> LRA_R
- U8 pad 2: IMU0_CS -> BTN_PWR
- U8 pad 3: LADC_CS -> unconnected-(U8-GPIO1-Pad3)
- U8 pad 34: I2C_SDA -> I2C1_SDA
- U8 pad 35: I2C_SCL -> I2C1_SCL
- U8 pad 36: USB_EN -> I2C0_SDA
- U8 pad 37: USB_SEL -> I2C0_SCL
- U8 pad 38: ESP_EN -> ADC_MUX_OUT
- U8 pad 4: IMU1_CS -> WL_ON
- U8 pad 5: LRA_L -> WL_D
- U8 pad 6: SPI_RX -> WL_CLK
- U8 pad 7: BTN_PWR -> WL_CS
- U8 pad 8: SPI_CK -> unconnected-(U8-GPIO6-Pad8)
- U8 pad 9: SPI_TX -> unconnected-(U8-GPIO7-Pad9)
Routing:
- net (no net): track 0.00 -> 119.0 mm
- net SPI_RX: track 103.8 -> 0.00 mm, vias 4 -> 0
- net SPI_TX: track 101.2 -> 0.00 mm, vias 6 -> 0
- net SPI_CK: track 99.5 -> 0.00 mm, vias 5 -> 0
- net RADC_CS: track 66.9 -> 0.00 mm, vias 3 -> 0
- net ESP_EN: track 64.8 -> 0.00 mm, vias 4 -> 0
- net I2C0_SCL: track 0.00 -> 51.0 mm, vias 0 -> 3
- net ADC_MUX_OUT: track 0.00 -> 48.9 mm, vias 0 -> 3
- net I2C0_SDA: track 0.00 -> 42.9 mm, vias 0 -> 3
- net PLAYER_RGB: track 41.4 -> 0.00 mm
- net UART_USB+: track 41.2 -> 0.00 mm, vias 2 -> 0
- net UART_USB-: track 40.7 -> 0.00 mm, vias 2 -> 0
- net LRA_R: track 66.5 -> 105.8 mm, vias 2 -> 3
- net Net-(P1A-DO): track 0.00 -> 36.2 mm, vias 0 -> 2
- net ESP_RTS: track 36.2 -> 0.00 mm, vias 2 -> 0
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
Commit message: More routing
Parts:
- moved R18 61.0 mm to (205.9, 126.5)
- moved R19 59.7 mm to (203.1, 126.5)
- moved S7 54.2 mm to (205.5, 116.3)
- moved U2 49.7 mm to (219.6, 95.1), turned to 90 degrees
- moved U3 48.7 mm to (221.8, 95.1), turned to 90 degrees
- moved L7 47.7 mm to (214.2, 108.5), turned to 90 degrees
- moved C18 42.7 mm to (181.5, 88.0)
- moved R8 31.1 mm to (234.1, 116.3), turned to 180 degrees
- moved R9 23.9 mm to (234.1, 115.6), turned to 0 degrees
- moved R17 17.5 mm to (205.2, 113.1)
- moved U1 15.1 mm to (216.5, 97.0), turned to -90 degrees
- moved R16 14.8 mm to (205.2, 112.4)
- moved U10 7.76 mm to (201.7, 123.8)
- moved U5 7.76 mm to (206.4, 123.8)
- moved C12 7.58 mm to (204.3, 121.6)
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Connections:
- Q3 pad 3: N_LATCH_3.3 -> N_DATA_3.3
- Q3 pad 4: N_LATCH_SAFE -> N_DATA_SAFE
- Q4 pad 3: N_DATA_3.3 -> N_LATCH_3.3
- Q4 pad 4: N_DATA_SAFE -> N_LATCH_SAFE
- R23 pad 2: N_LATCH_3.3 -> N_DATA_3.3
- R25 pad 2: N_DATA_3.3 -> N_LATCH_3.3
- R26 pad 2: N_LATCH_SAFE -> N_DATA_SAFE
- R28 pad 2: N_DATA_SAFE -> N_LATCH_SAFE
- U1 pad 5: VBUS_PRE -> +5V_PRE
- U11 pad B1: I2C_SCL -> I2C1_SCL
- U11 pad C1: I2C_SDA -> I2C1_SDA
- U2 pad 1: N_LATCH_SAFE -> N_CLOCK_SAFE
- U2 pad 3: N_CLOCK_SAFE -> N_LATCH_SAFE
- U2 pad 4: N_CLOCK -> N_LATCH
- U2 pad 6: N_LATCH -> N_CLOCK
- U3 pad 1: N_DATA_SAFE -> unconnected-(U3-I/O1-Pad1)
- U3 pad 3: unconnected-(U3-I/O2-Pad3) -> N_DATA_SAFE
- U3 pad 4: unconnected-(U3-I/O2-Pad4) -> N_DATA
- U3 pad 5: +3.3V_PRE -> +3V3_PRE
- U3 pad 6: N_DATA -> unconnected-(U3-I/O1-Pad6)
- U8 pad 2: BTN_PWR -> WL_ON
- U8 pad 3: unconnected-(U8-GPIO1-Pad3) -> WL_D
- U8 pad 30: N_LATCH_3.3 -> N_DATA_3.3
- U8 pad 31: N_DATA_3.3 -> N_LATCH_3.3
- U8 pad 38: ADC_MUX_OUT -> ZR_ANALOG
- U8 pad 39: RGB_OUT -> ZL_ANALOG
- U8 pad 4: WL_ON -> WL_CLK
- U8 pad 40: ZR_ANALOG -> RGB_OUT
- U8 pad 41: ZL_ANALOG -> ADC_MUX_OUT
- U8 pad 5: WL_D -> WL_CS
- U8 pad 6: WL_CLK -> ADC_ADDR_0
- U8 pad 7: WL_CS -> ADC_ADDR_1
- U8 pad 8: unconnected-(U8-GPIO6-Pad8) -> BTN_PWR
Routing:
- net (no net): track 119.0 -> 0.00 mm
- net LRA_R: track 105.8 -> 28.8 mm, vias 3 -> 1
- net +3V3: track 176.5 -> 132.7 mm
- net BAT_LVL: track 45.6 -> 7.08 mm, vias 2 -> 1
- net I2C_SDA: track 34.6 -> 0.00 mm, vias 3 -> 0
- net WL_CLK: track 3.33 -> 36.6 mm, vias 0 -> 2
- net I2C_SCL: track 32.7 -> 0.00 mm, vias 2 -> 0
- net WL_D: track 2.97 -> 35.4 mm, vias 0 -> 2
- net unconnected-(U8-GPIO1-Pad3): track 30.7 -> 0.00 mm, vias 1 -> 0
- net Net-(P1A-DO): track 36.2 -> 10.7 mm
- net WL_GP1: track 25.0 -> 0.00 mm, vias 2 -> 0
- net ADC_ADDR_0: track 0.00 -> 23.2 mm
- net WL_CS: track 2.30 -> 25.1 mm
- net ADC_MUX_OUT: track 48.9 -> 27.1 mm, vias 3 -> 2
- net WL_GP2: track 21.6 -> 0.00 mm, vias 2 -> 0
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Other:
- board text added: "GCU R5 Designed by Mitch 2.7.2025"
- board text removed: "GCU R4K Designed by Mitch 10.25.2024"

Commit message: Finalize Routing
Parts:
- moved C18 40.1 mm to (208.2, 117.9), turned to 0 degrees
- moved C13 3.32 mm to (202.1, 121.3), turned to -90 degrees
- moved R18 0.15 mm to (205.7, 126.5)
Routing:
- net RY: track 11.1 -> 90.6 mm
- net RX: track 10.0 -> 88.2 mm
- net LRA_R: track 28.8 -> 70.1 mm, vias 1 -> 2
- net I2C1_SCL: track 20.0 -> 24.1 mm
- net I2C1_SDA: track 18.4 -> 22.3 mm
- net +3V3: track 132.7 -> 135.3 mm
- net LRA_L: track 71.4 -> 73.5 mm
- net Net-(D4A-A): track 64.2 -> 62.4 mm
- net G: track 163.7 -> 165.3 mm
- net BTN_PWR: track 63.9 -> 62.3 mm
- net RP_RUN: track 61.6 -> 60.7 mm
- net I2C0_SDA: track 46.2 -> 46.5 mm, vias 3 -> 4
- net I2C0_SCL: track 45.7 -> 45.9 mm, vias 3 -> 5
- net X5: track 59.0 -> 59.2 mm, vias 3 -> 4
- net GND: vias 104 -> 127
