File: HW/Projects/Main_S1/UGC_Main_S1.kicad_sch (KiCad schematic)
At the start: 137 parts, among them J1 SM02B-SURS-TF_LF__SN_, J10 SM02B-SURS-TF_LF__SN_, J13 503480-0640, J2 503480-0640, J4 Conn_01x06_Pin, J5 UJ31-CH-G1-SMT-TR, J6 Trigger, J7 Trigger, J8 Conn_01x02, J9 Conn_01x02, Q3 BSS138DW, Q4 BSS138DW, Q5 MMBT2222A, Q6 MMBT2222A, SW1 SW_Push, SW10 SW_Push, SW11 SW_Push, SW12 SW_Push, SW13 SW_Push, SW14 TS-1187A-C-A-B, SW17 TS-1187A-C-A-B, SW18 TS-1187A-C-A-B, SW19 TS-1187A-C-A-B, SW2 SW_Push, SW3 SW_Push, SW4 SW_Push, SW5 TS-1187A-C-A-B, SW6 GL18_SW, SW7 SW_Push, SW8 SW_Push, SW9 TS-1187A-C-A-B, U1 ST_LSM6, U10 ST_LSM6, U2 GD25Q80EEIGR, U2 USBLC6-2P6, U3 USBLC6-2P6, U4 TPS630001RCR, U5 USBLC6-2P6, U8 RP2040, X1 ModConnect, X2 ModConnect, X3 ModConnect, X4 ModConnect, X5 ModConnect, X6 ModConnect, Y1 ABM8-272-T3

Commit message: S1 Version PCB Updates
Parts:
- removed J13: 503480-0640, hhl:5034800640, symbol hhl:503480-0640
- removed J4: Conn_01x06_Pin, Connector_PinHeader_2.00mm:PinHeader_1x06_P2.00mm_Vertical, symbol Connector:Conn_01x06_Pin
- removed J5: UJ31-CH-G1-SMT-TR, hhl:CUI_UJ31-CH-G1-SMT-TR, symbol hhl:UJ31-CH-G1-SMT-TR
- added C17: 1uF, Capacitor_SMD:C_0402_1005Metric, symbol Device:C
- added J11: USB4056-03-A2, hhl:USB405603A, symbol hhl:USB4056-03-A
- added J3: Molex 5051100792, hhl:CON_5051100792_MOL, symbol Connector:Conn_01x07_Pin
- added L14, L15, L16, L17, L18, L7, L8, L9: SK6805-EC-10, hhl:SK6805-EC-10, symbol hhl:SK6805-EC-10
- SW1, SW2, SW3, SW4: footprint hhl:ring_pad -> hhl:pgs_abxy
- SW10, SW11, SW12, SW13: footprint hhl:ring_dpad -> hhl:pgs_dpad
- SW14, SW17, SW18, SW19, SW5, SW9: value TS-1187A-C-A-B -> TS-1187A-C-A-B
- renumbered C10 to C11, C3 to C23, C1 to C3, C2 to C4, D1 to D4, D2 to D5, R7 to R10, U2 to U9
Connections:
- net +1V1: now also C17.2
- net +3V3: now also J3.6 (Pin_6), L14.2 (VDD), L15.2 (VDD), L16.2 (VDD), L17.2 (VDD), L18.2 (VDD), L7.2 (VDD), L8.2 (VDD), L9.2 (VDD)
- net +3V3_PRE: now also J11.A2 (SSTXP1), J11.B2 (SSTXP2)
- net ABXY_RGB: now also L7.1 (DIN)
- net CC1: now also J11.A5 (CC1)
- net CC2: now also J11.B5 (CC2)
- net D+: now also J11.A6 (DP1), J11.B6 (DP2)
- net D-: now also J11.A7 (DN1), J11.B7 (DN2)
- net GND: now also C17.1, J11.A1 (GND_1), J11.A12 (GND_2), J11.B1 (GND_3), J11.B12 (GND_4), J11.MH1, J11.MH2, J11.MH3, J11.MH4, J3.1 (Pin_1), L14.4 (GND), L15.4 (GND), L16.4 (GND), L17.4 (GND), L18.4 (GND), L7.4 (GND), L8.4 (GND), L9.4 (GND)
- net NC: now also L14.3 (DOUT); no longer L13.3 (DOUT)
- net N_CLOCK: now also J11.A3 (SSTXN1), J11.B3 (SSTXN2)
- net N_DATA: now also J11.A11 (SSRXP2), J11.B11 (SSRXP1)
- net N_LATCH: now also J11.A10 (SSRXN2), J11.B10 (SSRXN1)
- net PLAYER_RGB: now also L18.3 (DOUT); no longer L4.3 (DOUT)
- net RS_B_IN: now also J3.3 (Pin_3)
- net RS_B_OUT: now also J3.2 (Pin_2)
- net RX: now also J3.5 (Pin_5)
- net RY: now also J3.4 (Pin_4)
- net VBUS_SYS: now also J11.A4 (VBUS_1), J11.A9 (VBUS_2), J11.B4 (VBUS_3), J11.B9 (VBUS_4)
- net LED1: now reaches L10.3 (DOUT), L11.1 (DIN)
- net LED1: now also L8.1 (DIN)
- net LED2: now reaches L11.3 (DOUT), L12.1 (DIN)
- net LED2: now also L9.1 (DIN)
- net LED3: now reaches L12.3 (DOUT), L13.1 (DIN)
- net LED3: now also L14.1 (DIN)
- new net: L15.3 (DOUT), L16.1 (DIN)
- new net: L16.3 (DOUT), L17.1 (DIN)
- new net: L17.3 (DOUT), L18.1 (DIN)
- new net DPAD_RGB: L15.1 (DIN), L4.3 (DOUT)
- new net RGB_OUT_CSTICK: J3.7 (Pin_7), L13.3 (DOUT)
Other:
- note added: "C17 must be near pin 45"
- note added: "C8 must be near pin 44"

Commit message: GCU R5 Update
- Add fuel gauge IC
Parts:
- L1, L10, L11, L12, L13, L14, L15, L16, L17, L18, L2, L3, L4, L6, L7, L8, L9: LCSC C2890035 -> (none)
Other:
- note added: "idx 0"
- note added: "idx 1"
- note added: "idx 10 (Y)"
- note added: "idx 11 (A)"
- note added: "idx 12 (X)"
- note added: "idx 2"
- note added: "idx 3"
- note added: "idx 4 (left)"
- note added: "idx 5 (down)"
- note added: "idx 6 (right)"
- note added: "idx 7 (up)"
- note added: "idx 8"
- note added: "idx 9 (B)"
- note added: "right stick idx 13 idx 14 idx 15 idx 16"
Changed lines of the file:
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@@
 		)
 	)
+	(text "idx 1"
+		(exclude_from_sim no)
+		(at 299.72 101.6 0)
+		(effects
+			(font
+				(size 1.27 1.27)
+			)
+		)
+	)
 	(text "DL"
 		(exclude_from_sim no)
@@
 		)
 	)
+	(text "idx 12 (X)"
+		(exclude_from_sim no)
+		(at 345.694 159.004 0)
+		(effects
+			(font
+				(size 1.27 1.27)
+			)
+		)
+	)
 	(text "USB I/O"
 		(exclude_from_sim no)
@@
 		)
 	)
+	(text "idx 8"
+		(exclude_from_sim no)
+		(at 276.86 137.922 0)
+		(effects
+			(font
+				(size 1.27 1.27)
+			)
+		)
+	)
+	(text "idx 10 (Y)"
+		(exclude_from_sim no)
+		(at 299.72 158.75 0)
+		(effects
+			(font
+				(size 1.27 1.27)
+			)
+		)
+	)
+	(text "idx 9 (B)"
+		(exclude_from_sim no)
+		(at 276.86 159.004 0)
+		(effects
+			(font
+				(size 1.27 1.27)
+			)
+		)
+	)
 	(text "Fn"
 		(exclude_from_sim no)
@@
 		)
 	)
+	(text "idx 0"
+		(exclude_from_sim no)
+		(at 276.86 101.6 0)
+		(effects
+			(font
+				(size 1.27 1.27)
+			)
+		)
+	)
 	(text "IMU 1"
 		(exclude_from_sim no)
@@
 		)
 	)
+	(text "idx 2"
+		(exclude_from_sim no)
+		(at 322.834 101.6 0)
+		(effects
+			(font
+				(size 1.27 1.27)
+			)
+		)
+	)
+	(text "idx 4 (left)"
+		(exclude_from_sim no)
+		(at 249.682 176.784 0)
+		(effects
+			(font
+				(size 1.27 1.27)
+			)
+		)
+	)
 	(text "Flash"
 		(exclude_from_sim no)
@@
 		)
 	)
+	(text "right stick\nidx 13\nidx 14\nidx 15\nidx 16"
+		(exclude_from_sim no)
+		(at 363.474 132.334 0)
+		(effects
+			(font
+				(size 1.27 1.27)
+			)
+		)
+	)
+	(text "idx 11 (A)"
+		(exclude_from_sim no)
+		(at 322.58 158.75 0)
+		(effects
+			(font
+				(size 1.27 1.27)
+			)
+		)
+	)
 	(text "DD"
 		(exclude_from_sim no)
@@
 		)
 	)
+	(text "idx 3"
+		(exclude_from_sim no)
+		(at 345.44 102.108 0)
+		(effects
+			(font
+				(size 1.27 1.27)
+			)
+		)
+	)
 	(text "Y"
 		(exclude_from_sim no)
@@
 		)
 	)
+	(text "idx 6 (right)"
+		(exclude_from_sim no)
+		(at 250.698 129.794 0)
+		(effects
+			(font
+				(size 1.27 1.27)
+			)
+		)
+	)
 	(text "3.3 Regulation"
 		(exclude_from_sim no)
@@
 		)
 	)
+	(text "idx 5 (down)"
+		(exclude_from_sim no)
+		(at 250.698 154.178 0)
+		(effects
+			(font
+				(size 1.27 1.27)
+			)
+		)
+	)
 	(text "Analog\nTriggers"
 		(exclude_from_sim no)
@@
 		)
 	)
+	(text "idx 7 (up)"
+		(exclude_from_sim no)
+		(at 249.682 108.458 0)
+		(effects
+			(font
+				(size 1.27 1.27)
+			)
+		)
+	)
 	(text "ZL"
 		(exclude_from_sim no)
@@
 			)
 		)
-		(property "LCSC" "C2890035"
+		(property "LCSC" ""
 			(at 276.86 130.81 0)
 			(effects
@@
 			)
 		)
-		(property "LCSC" "C2890035"
+		(property "LCSC" ""
 			(at 276.86 186.69 0)
 			(effects
@@
 			)
 		)
-		(property "LCSC" "C2890035"
+		(property "LCSC" ""
 			(at 238.76 176.53 0)
 			(effects
@@
 			)
 		)
-		(property "LCSC" "C2890035"
+		(property "LCSC" ""
 			(at 238.76 130.81 0)
 			(effects
@@
 			)
 		)
-		(property "LCSC" "C2890035"
+		(property "LCSC" ""
 			(at 276.86 101.6 0)
 			(effects
@@
 			)
 		)
-		(property "LCSC" "C2890035"
+		(property "LCSC" ""
 			(at 322.58 186.69 0)
 			(effects
@@
 			)
 		)
-		(property "LCSC" "C2890035"
+		(property "LCSC" ""
 			(at 299.72 158.75 0)
 			(effects
@@
 			)
 		)
-		(property "LCSC" "C2890035"
+		(property "LCSC" ""
 			(at 345.44 101.6 0)
 			(effects
@@
 			)
 		)
-		(property "LCSC" "C2890035"
+		(property "LCSC" ""
 			(at 345.44 158.75 0)
 			(effects
@@
 			)
 		)
-		(property "LCSC" "C2890035"
+		(property "LCSC" ""
 			(at 276.86 158.75 0)
 			(effects
@@
 			)
 		)
-		(property "LCSC" "C2890035"
+		(property "LCSC" ""
 			(at 345.44 186.69 0)
 			(effects
@@
 			)
 		)
-		(property "LCSC" "C2890035"
+		(property "LCSC" ""
 			(at 238.76 107.95 0)
 			(effects
@@
 			)
 		)
-		(property "LCSC" "C2890035"
+		(property "LCSC" ""
 			(at 322.58 101.6 0)
 			(effects
@@
 			)
 		)
-		(property "LCSC" "C2890035"
+		(property "LCSC" ""
 			(at 299.72 186.69 0)
 			(effects
@@
 			)
 		)
-		(property "LCSC" "C2890035"
+		(property "LCSC" ""
 			(at 299.72 101.6 0)
 			(effects
@@
 			)
 		)
-		(property "LCSC" "C2890035"
+		(property "LCSC" ""
 			(at 238.76 153.67 0)
 			(effects
@@
 			)
 		)
-		(property "LCSC" "C2890035"
+		(property "LCSC" ""
 			(at 322.58 158.75 0)
 			(effects

Commit message: PCB Updates
- Change potentiometer orientation for trigger sliders
Connections:
- net +3V3: now also R37.1, R4.1, S3.1 (Pin_1), S6.1 (Pin_1); no longer R36.2, R38.2, S1.1 (Pin_1), S4.1 (Pin_1)
- net GND: now also R36.2, R38.2, S1.1 (Pin_1), S4.1 (Pin_1); no longer R37.1, R4.1, S3.1 (Pin_1), S6.1 (Pin_1)

Commit message: Updates
Parts:
- added D1: CUS08F30,H3F, Diode_SMD:D_SOD-323_HandSoldering, symbol progcc_v3:CUS08F30
- added J5: Conn_01x05_Socket, Connector_Molex:Molex_PicoBlade_53261-0571_1x05-1MP_P1.25mm_Horizontal, symbol Connector:Conn_01x05_Socket
- added R13, R14, R15, R16, R17, R18, R19, R20, R29, R30, R8, R9: 100R, Resistor_SMD:R_0201_0603Metric, symbol Device:R
- R3, R32, R40: footprint Resistor_SMD:R_0402_1005Metric -> Resistor_SMD:R_0201_0603Metric; LCSC C106232 -> C77623; MPN RC0402FR-07100RL -> RC0201FR-07100RL; Package 0402 -> 0201
Connections:
- net A: now also R14.1
- net B: now also R15.1
- net C: now also R16.1
- net D: now also R17.1
- net GND: now also J5.4 (Pin_4), J5.5 (Pin_5)
- net N_CLOCK_3.3: now also R13.2; no longer U8.32 (GPIO21)
- net N_DATA_3.3: now also R9.2; no longer U8.31 (GPIO20)
- net N_LATCH_3.3: now also R8.2; no longer U8.30 (GPIO19)
- net SAFE_D+: now also J5.3 (Pin_3)
- net SAFE_D-: now also J5.2 (Pin_2)
- net VBUS_SYS: now also D1.1 (K); no longer J11.A4 (VBUS_1), J11.A9 (VBUS_2), J11.B4 (VBUS_3), J11.B9 (VBUS_4), U2.5 (VBUS)
- new net: R8.1, U8.30 (GPIO19)
- new net: R9.1, U8.31 (GPIO20)
- new net: R13.1, U8.32 (GPIO21)
- new net A_GPIO: R14.2
- new net B_GPIO: R15.2
- new net C_GPIO: R16.2
- new net D_GPIO: R17.2
- new net E_GPIO: R18.2
- new net F_GPIO: R19.2
- new net G_GPIO: R20.2
- new net H_GPIO: R29.2
- new net I_GPIO: R30.2
- new net VBUS: D1.2 (A), J11.A4 (VBUS_1), J11.A9 (VBUS_2), J11.B4 (VBUS_3), J11.B9 (VBUS_4), J5.1 (Pin_1), U2.5 (VBUS)

Commit message: R5/S1 Updates
Parts:
- removed J6, J7: Trigger, Connector_JST:JST_PH_B2B-PH-K_1x02_P2.00mm_Vertical, symbol Connector:Conn_01x02_Pin
- removed R17, R18, R19, R20, R29, R30: 100R, Resistor_SMD:R_0201_0603Metric, symbol Device:R
- removed R36, R37, R38, R4: 75k, Resistor_SMD:R_0402_1005Metric, symbol Device:R
- removed RV1, RV2: Slider_GCC-Gamecube_MB, hhl:GCC_Slider_MillMaxSocketed, symbol hhl:Slider_GCC-Gamecube_SolderInsert
- removed S1, S2, S3, S4, S5, S6: 4015-0-43-80-30-27-10-0, hhl:4015-0-43-80-30-27-10-0, symbol Connector:Conn_01x01_Socket
- added J6, J9: Conn_01x04_Socket, hhl:5051100492, symbol Connector:Conn_01x04_Socket
- renumbered C12 to C1, C26 to C10, C27 to C11, C3 to C12, C4 to C13, C24 to C14, C5 to C15, C17 to C16, C14 to C17, C15 to C18, C6 to C19, C13 to C2, C7 to C20, C8 to C21, C23 to C22, C9 to C23, C10 to C24, C11 to C25, C2 to C3, C1 to C4, C16 to C5, C32 to C6, C25 to C7, C33 to C8, C34 to C9, D3 to D1, D12 to D10, D13 to D11, D11 to D12, D8 to D13, D4 to D14, D5 to D15, D14 to D2, D6 to D3, D7 to D4, D15 to D5, D16 to D6, D9 to D7, D10 to D8, D1 to D9, J11 to J1, J2 to J10, J3 to J2, J5 to J3, J1 to J4, J10 to J5, J9 to J7, L18 to L1, L11 to L10, L8 to L11, L5 to L12, L3 to L13, L12 to L14, L9 to L15, L4 to L16, L13 to L17, L14 to L18, L17 to L2, L16 to L3, L15 to L4, L1 to L5, L10 to L7, L7 to L8, L2 to L9, Q3 to Q1, Q4 to Q2, Q5 to Q3, Q6 to Q4, R23 to R1, R1 to R10, R31 to R11, R39 to R12, R32 to R13, R40 to R14, R33 to R15, R41 to R16, R5 to R17, R3 to R18, R6 to R19, R24 to R2, R7 to R20, R11 to R21, R12 to R22, R14 to R23, R15 to R24, R16 to R25, R8 to R26, R9 to R27, R13 to R28, R35 to R29, R25 to R3, R34 to R30, R10 to R31, R26 to R4, R27 to R5, R28 to R6, R2 to R7, R21 to R8, R22 to R9, S7 to S1, SW6 to SW1, SW12 to SW10, SW7 to SW11, SW1 to SW12, SW3 to SW13, SW4 to SW14, SW8 to SW15, SW5 to SW16, SW14 to SW17, SW9 to SW2, SW17 to SW3, SW18 to SW4, SW19 to SW5, SW13 to SW6, SW2 to SW7, SW10 to SW8, SW11 to SW9, TP6 to TP1, TP1 to TP2, TP7 to TP3, TP2 to TP4, U10 to U2, U2 to U3, U3 to U4, U4 to U6, U8 to U7, U9 to U8, X6 to X2, X5 to X3, X2 to X4, X3 to X5, X4 to X6
Connections:
- net A_GPIO is gone; now on net I: R23.2
- net B_GPIO is gone; now on net H: R24.2
- net C_GPIO is gone; now on net G: R25.2
- net +3V3: now also J6.1 (Pin_1), J9.1 (Pin_1)
- net A: no longer R23.1
- net B: no longer R24.1
- net C: no longer R25.1
- net G: now also J8.1 (Pin_1); no longer J8.2 (Pin_2), U7.15 (GPIO12)
- net GND: now also J6.3 (Pin_3), J6.4 (Pin_4), J9.3 (Pin_3), J9.4 (Pin_4)
- net H: now also J7.1 (Pin_1); no longer J7.2 (Pin_2), U7.14 (GPIO11)
- net I: no longer U7.13 (GPIO10)
- net LS_BTN_IN: no longer J7.1 (Pin_1)
- net ZL_ANALOG: now also J6.2 (Pin_2)
- net ZR_ANALOG: now also J9.2 (Pin_2)
- net at D14.1 (A), R30.1: no longer J8.1 (Pin_1)
- net at D15.3 (A): now also J8.2 (Pin_2)
- net at D12.3 (A): now also J7.2 (Pin_2)
- new net: R24.1, U7.14 (GPIO11)
- new net: R23.1, U7.13 (GPIO10)
- new net: R25.1, U7.15 (GPIO12)
Other:
- note removed: "L"
- note removed: "R"
- moved on the sheet: J7, J8, R23, R24, R25

Commit message: Prod Update
Parts:
- added R32: 100k, Resistor_SMD:R_0402_1005Metric, symbol Device:R_Small
- J3: LCSC (none) -> C17256390
- R26, R27, R28: value 100R -> 27R; LCSC C77623 -> C273268; MPN RC0201FR-07100RL -> RC0201FR-0727RL
Connections:
- net +3V3_PRE: now also R32.2
- net GND: now also R32.1
Changed lines of the file:
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@@
 	)
 	(junction
+		(at 270.51 53.34)
+		(diameter 0)
+		(color 0 0 0 0)
+	)
+	(junction
 		(at 43.18 166.37)
 		(diameter 0)
@@
 	)
 	(junction
-		(at 107.95 118.11)
+		(at 246.38 99.06)
 		(diameter 0)
 		(color 0 0 0 0)
 	)
 	(junction
-		(at 246.38 99.06)
+		(at 91.44 166.37)
 		(diameter 0)
 		(color 0 0 0 0)
 	)
 	(junction
-		(at 91.44 166.37)
+		(at 411.48 248.92)
 		(diameter 0)
 		(color 0 0 0 0)
 	)
 	(junction
-		(at 411.48 248.92)
+		(at 259.08 57.15)
 		(diameter 0)
 		(color 0 0 0 0)
@@
 	)
 	(junction
-		(at 95.25 118.11)
-		(diameter 0)
-		(color 0 0 0 0)
-	)
-	(junction
 		(at 387.35 237.49)
 		(diameter 0)
@@
 	(wire
 		(pts
-			(xy 257.81 57.15) (xy 260.35 57.15)
+			(xy 257.81 57.15) (xy 259.08 57.15)
 		)
 		(stroke
@@
 	(wire
 		(pts
+			(xy 259.08 57.15) (xy 260.35 57.15)
+		)
+		(stroke
+			(width 0)
+			(type default)
+		)
+	)
+	(wire
+		(pts
 			(xy 134.62 45.72) (xy 133.35 45.72)
 		)
@@
 	(wire
 		(pts
-			(xy 280.67 38.1) (xy 283.21 38.1)
-		)
-		(stroke
-			(width 0)
-			(type default)
-		)
-	)
-	(wire
-		(pts
 			(xy 388.62 349.25) (xy 387.35 350.52)
 		)
@@
 	(wire
 		(pts
-			(xy 106.68 118.11) (xy 107.95 118.11)
-		)
-		(stroke
-			(width 0)
-			(type default)
-		)
-	)
-	(wire
-		(pts
 			(xy 290.83 146.05) (xy 290.83 156.21)
 		)
@@
 		)
 	)
+	(wire
+		(pts
+			(xy 259.08 53.34) (xy 259.08 57.15)
+		)
+		(stroke
+			(width 0)
+			(type default)
+		)
+	)
 	(polyline
 		(pts
@@
 	(wire
 		(pts
+			(xy 283.21 34.29) (xy 283.21 38.1)
+		)
+		(stroke
+			(width 0)
+			(type default)
+		)
+	)
+	(wire
+		(pts
 			(xy 236.22 142.24) (xy 241.3 142.24)
 		)
@@
 		)
 	)
+	(wire
+		(pts
+			(xy 270.51 53.34) (xy 270.51 57.15)
+		)
+		(stroke
+			(width 0)
+			(type default)
+		)
+	)
 	(polyline
 		(pts
@@
 	(wire
 		(pts
-			(xy 270.51 53.34) (xy 270.51 57.15)
+			(xy 270.51 50.8) (xy 270.51 53.34)
 		)
 		(stroke
@@
 	(wire
 		(pts
+			(xy 266.7 53.34) (xy 270.51 53.34)
+		)
+		(stroke
+			(width 0)
+			(type default)
+		)
+	)
+	(wire
+		(pts
 			(xy 92.71 176.53) (xy 92.71 187.96)
 		)
@@
 	(wire
 		(pts
+			(xy 261.62 53.34) (xy 259.08 53.34)
+		)
+		(stroke
+			(width 0)
+			(type default)
+		)
+	)
+	(wire
+		(pts
 			(xy 387.35 163.83) (xy 387.35 152.4)
 		)
@@
 	(wire
 		(pts
-			(xy 96.52 118.11) (xy 95.25 118.11)
-		)
-		(stroke
-			(width 0)
-			(type default)
-		)
-	)
-	(wire
-		(pts
 			(xy 133.35 58.42) (xy 134.62 58.42)
 		)
@@
 	(global_label "+3V3_PRE"
 		(shape input)
-		(at 270.51 53.34 90)
+		(at 270.51 50.8 90)
 		(fields_autoplaced yes)
 		(effects
@@
 		)
 		(property "Intersheetrefs" "${INTERSHEET_REFS}"
-			(at 270.51 40.6182 90)
+			(at 270.51 38.0782 90)
 			(effects
 				(font
@@
 	(global_label "VBUS_SYS"
 		(shape input)
-		(at 280.67 38.1 180)
+		(at 283.21 34.29 0)
 		(fields_autoplaced yes)
 		(effects
@@
 				(size 1.27 1.27)
 			)
-			(justify right)
+			(justify left)
 		)
 		(property "Intersheetrefs" "${INTERSHEET_REFS}"
-			(at 268.311 38.1 0)
+			(at 295.569 34.29 0)
 			(effects
 				(font
 					(size 1.27 1.27)
 				)
-				(justify right)
+				(justify left)
 				(hide yes)
 			)
@@
 			)
 		)
-		(property "Description" "Custom right angle silicone tactile switch 5mm button height"
+		(property "Description" "Custom right angle silicone tactile switch 3.85mm button height"
 			(at 402.59 173.99 0)
 			(effects
@@
 			)
 		)
-		(property "Description" "Custom right angle silicone tactile switch 5mm button height"
+		(property "Description" "Custom right angle silicone tactile switch 3.85mm button height"
 			(at 402.59 280.67 0)
 			(effects
@@
 			)
 		)
-		(property "Value" "100R"
+		(property "Value" "27R"
 			(at 356.87 331.47 90)
 			(effects
@@
 			)
 		)
-		(property "Description" "62.5mW Thick Film Resistors 50V ±100ppm/℃ ±1% 100Ω"
+		(property "Description" "50mW Thick Film Resistors 25V ±1% ±200ppm/℃ 27Ω"
 			(at 356.87 331.47 0)
 			(effects
@@
 			)
 		)
-		(property "LCSC" "C77623"
+		(property "LCSC" "C273268"
 			(at 356.87 331.47 0)
 			(effects
@@
 			)
 		)
-		(property "MPN" "RC0201FR-07100RL"
+		(property "MPN" "RC0201FR-0727RL "
 			(at 356.87 331.47 0)
 			(effects
@@
 	)
 	(symbol
+		(lib_id "Device:R_Small")
+		(at 264.16 53.34 90)
+		(unit 1)
+		(exclude_from_sim no)
+		(in_bom yes)
+		(on_board yes)
+		(dnp no)
+		(property "Reference" "R32"
+			(at 264.16 49.784 90)
+			(effects
+				(font
+					(size 1.27 1.27)
+				)
+			)
+		)
+		(property "Value" "100k"
+			(at 264.16 51.562 90)
+			(effects
+				(font
+					(size 1.27 1.27)
+				)
+			)
+		)
+		(property "Footprint" "Resistor_SMD:R_0402_1005Metric"
+			(at 264.16 53.34 0)
+			(effects
+				(font
+					(size 1.27 1.27)
+				)
+				(hide yes)
+			)
+		)
+		(property "Datasheet" "~"
+			(at 264.16 53.34 0)
+			(effects
+				(font
+					(size 1.27 1.27)
+				)
+				(hide yes)
+			)
+		)
+		(property "Description" "100kΩ 62.5mW 50V Thick Film Resistor ±100ppm/℃ ±1% 0402 Chip Resistor - Surface Mount RoHS"
+			(at 264.16 53.34 0)
+			(effects
+				(font
+					(size 1.27 1.27)
+				)
+				(hide yes)
+			)
+		)
+		(property "JLCPN" ""
+			(at 264.16 53.34 0)
+			(effects
+				(font
+					(size 1.27 1.27)
+				)
+				(hide yes)
+			)
+		)
+		(property "LCSC" "C60491"
+			(at 264.16 53.34 0)
+			(effects
+				(font
+					(size 1.27 1.27)
+				)
+				(hide yes)
+			)
+		)
+		(property "MPN" "RC0402FR-07100KL"
+			(at 264.16 53.34 0)
+			(effects
+				(font
+					(size 1.27 1.27)
+				)
+				(hide yes)
+			)
+		)
+		(property "Price" "0.0004"
+			(at 264.16 53.34 0)
+			(effects
+				(font
+					(size 1.27 1.27)
+				)
+				(hide yes)
+			)
+		)
+		(property "Link" ""
+			(at 264.16 53.34 0)
+			(effects
+				(font
+					(size 1.27 1.27)
+				)
+				(hide yes)
+			)
+		)
+		(property "Package" "0402"
+			(at 264.16 53.34 0)
+			(effects
+				(font
+					(size 1.27 1.27)
+				)
+				(hide yes)
+			)
+		)
+		(pin "1"
+		)
+		(pin "2"
+		)
+		(instances
+			(project "UGC_Main_S1"
+				(path "/5d3b68ed-8c8a-4ed0-8f2b-63049c253646"
+					(reference "R32")
+					(unit 1)
+				)
+			)
+		)
+	)
+	(symbol
 		(lib_id "power:GND")
 		(at 179.07 110.49 270)
@@
 			)
 		)
-		(property "Value" "100R"
+		(property "Value" "27R"
 			(at 356.87 328.93 90)
 			(effects
@@
 			)
 		)
-		(property "Description" "62.5mW Thick Film Resistors 50V ±100ppm/℃ ±1% 100Ω"
+		(property "Description" "50mW Thick Film Resistors 25V ±1% ±200ppm/℃ 27Ω"
 			(at 356.87 328.93 0)
 			(effects
@@
 			)
 		)
-		(property "LCSC" "C77623"
+		(property "LCSC" "C273268"
 			(at 356.87 328.93 0)
 			(effects
@@
 			)
 		)
-		(property "MPN" "RC0201FR-07100RL"
+		(property "MPN" "RC0201FR-0727RL "
 			(at 356.87 328.93 0)
 			(effects
@@
 			)
 		)
+		(property "LCSC" "C17256390"
+			(at 163.83 54.61 0)
+			(effects
+				(font
+					(size 1.27 1.27)
+				)
+				(hide yes)
+			)
+		)
 		(pin "4"
 		)
@@
 			)
 		)
-		(property "Value" "100R"
+		(property "Value" "27R"
 			(at 356.87 326.39 90)
 			(effects
@@
 			)
 		)
-		(property "Description" "62.5mW Thick Film Resistors 50V ±100ppm/℃ ±1% 100Ω"
+		(property "Description" "50mW Thick Film Resistors 25V ±1% ±200ppm/℃ 27Ω"
 			(at 356.87 326.39 0)
 			(effects
@@
 			)
 		)
-		(property "LCSC" "C77623"
+		(property "LCSC" "C273268"
 			(at 356.87 326.39 0)
 			(effects
@@
 			)
 		)
-		(property "MPN" "RC0201FR-07100RL"
+		(property "MPN" "RC0201FR-0727RL "
 			(at 356.87 326.39 0)
 			(effects

Commit message: PCB Updates
Parts:
- removed TP1, TP2, TP3, TP4: TestPoint, TestPoint:TestPoint_Pad_2.0x2.0mm, symbol Connector:TestPoint

Commit message: PCB Prod Update
Parts:
- C1, C14, C15, C19, C2, C20, C23, C24, C25, C5, C6, C7: footprint Capacitor_SMD:C_0402_1005Metric -> Capacitor_SMD:C_0201_0603Metric; MPN CC0402KRX7R5BB104 -> CL03A104KQ3NNNC; Package 0402 -> 0201
- C10, C11, C16, C21, C8, C9: footprint Capacitor_SMD:C_0402_1005Metric -> Capacitor_SMD:C_0201_0603Metric; MPN CL05A105KQ5NNNC -> GRM033R60J105KEA2D; Package 0402 -> 0201
- C12: Package (none) -> CASE-A-3216-18(mm)
- R1, R10, R2, R22, R3, R31, R4, R5, R6, R7: footprint Resistor_SMD:R_0402_1005Metric -> Resistor_SMD:R_0201_0603Metric; MPN RC0402FR-071KL -> RC0201FR-071KL; Package 0402 -> 0201
- R11, R12, R17: footprint Resistor_SMD:R_0402_1005Metric -> Resistor_SMD:R_0201_0603Metric; MPN RC0402FR-0710KL -> RC0201FR-0710KL; Package 0402 -> 0201
- R15, R16, R29, R30: footprint Resistor_SMD:R_0402_1005Metric -> Resistor_SMD:R_0201_0603Metric; MPN RC0402FR-070RL -> RC0201FR-070RL; Package 0402 -> 0201
- R21: footprint Resistor_SMD:R_0402_1005Metric -> Resistor_SMD:R_0201_0603Metric; MPN RC0402FR-07330RL -> RC0201FR-07330RL; Package 0402 -> 0201
- R8, R9: footprint Resistor_SMD:R_0402_1005Metric -> Resistor_SMD:R_0201_0603Metric; MPN RC0402FR-075K1L -> RC0201FR-075K1L; Package 0402 -> 0201
