File: HW/Projects/Trigger Hall FPC/FPC_Trigger_Board.kicad_sch (KiCad schematic)
At the start: 8 parts, among them U1 HAL4395, U2 HAL4395

Commit message: R5/S1 Updates
Parts:
- removed JP1, JP2, JP3, JP4: SolderJumper_3_Bridged12, Jumper:SolderJumper-3_P1.3mm_Bridged12_RoundedPad1.0x1.5mm_NumberLabels, symbol Jumper:SolderJumper_3_Bridged12
- removed U1, U2: HAL4395, Package_TO_SOT_SMD:SOT-23-5, symbol hhl:HAL4395SO5
- added J1, J2: Conn_01x04_Pin, hhl:505110-0492 Ribbon, symbol Connector:Conn_01x04_Pin
- added U1, U2: HAL4395, hhl:SOT-23-5L, symbol Regulator_Linear:TLV70012_SOT23-5
Connections:
- net PAD_1L is gone; now on net +3V3L: C1.2
- net PAD_1R is gone; now on net +3V3: C2.2
- net PAD_2L is gone; now on net GNDL: C1.1
- net PAD_2R is gone; now on net GND: C2.1
- net +3V3: now also J2.1 (Pin_1), U2.1 (VCC)
- net +3V3L: now also J1.1 (Pin_1), U1.1 (VCC)
- net ADC_0: now also J1.2 (Pin_2), U1.5 (OUT)
- net ADC_1: now also J2.2 (Pin_2), U2.5 (OUT)
- net GND: now also J2.3 (Pin_3), J2.4 (Pin_4), U2.2 (~{EN}), U2.3 (GND)
- net GNDL: now also J1.3 (Pin_3), J1.4 (Pin_4), U1.2 (~{EN}), U1.3 (GND)
